File: sheets/power_rails.kicad_sch (KiCad schematic)
At the start: 0 parts

Commit message: sch: power rails (buck + LDOs + INA226 telemetry + ADC dividers)
Parts:
- added C33, C39: 0.1uF/16V, C_0603, symbol Device:C_Small
- added C34: 0.1uF/25V, C_0603, symbol Device:C_Small
- added C35, C36: 10uF/25V, C_1210, symbol Device:C_Small
- added C37, C38: 22uF/16V, C_1210, symbol Device:C_Small
- added C40, C41, C42, C43: 1uF/16V, C_0603, symbol Device:C_Small
- added D17, D18: B5819W, D_SOD-323, symbol Device:D_Schottky
- added L4: 2.2uH, L_8x8mm_H4mm, symbol Device:L_Small
- added R39, R44: 0.002/1W, R_1206, symbol Device:R_Small
- added R40: 1.00M, R_0603, symbol Device:R_Small
- added R41, R45, R47, R48, R49, R50: 100k, R_0603, symbol Device:R_Small
- added R42: 33.2k, R_0603, symbol Device:R_Small
- added R43, R46: 10.0k, R_0603, symbol Device:R_Small
- added U13, U14: INA226AIDGSR, Package_SO:MSOP-10_3x3mm_P0.5mm, symbol sierra-to-usb:INA226
- added U17: AP2112K-3.3TRG1, Package_TO_SOT_SMD:SOT-23-5, symbol Regulator_Linear:AP2112K-3.3
- added U3: TPS565201DDCR, Package_TO_SOT_SMD:SOT-23-6, symbol sierra-to-usb:TPS565201
- added U5: AP2112K-1.8TRG1, Package_TO_SOT_SMD:SOT-23-5, symbol Regulator_Linear:AP2112K-1.8
Connections:
- new net +12V: R39.1, R40.1, R45.1, U13.10 (IN+)
- new net +12V_BUCK: C35.1, C36.1, R39.2, U13.8 (VBUS), U13.9 (IN-), U3.3 (VIN)
- new net +1V8: C41.1, R49.1, U5.5 (VOUT)
- new net +3V3: C33.1, C37.1, C38.1, C39.1, C40.1, D18.2 (A), L4.2, R42.1, R44.1, R47.1, U13.6 (VS), U14.10 (IN+), U14.2 (A0), U14.6 (VS), U5.1 (VIN), U5.3 (EN)
- new net +3V3_MCU: C43.1, U17.5 (VOUT)
- new net +3V3_MOD: R44.2, U14.8 (VBUS), U14.9 (IN-)
- new net BUCK_EN: R40.2, R41.1, U3.5 (EN)
- new net GND: C33.2, C35.2, C36.2, C37.2, C38.2, C39.2, C40.2, C41.2, C42.2, C43.2, R41.2, R43.2, R46.2, R48.2, R50.2, U13.1 (A1), U13.2 (A0), U13.7 (GND), U14.1 (A1), U14.7 (GND), U17.2 (GND), U3.1 (GND), U5.2 (GND)
- new net I2C_SCL: U13.5 (SCL), U14.5 (SCL)
- new net I2C_SDA: U13.4 (SDA), U14.4 (SDA)
- new net N_OR17: C42.1, D17.1 (K), D18.1 (K), U17.1 (VIN), U17.3 (EN)
- new net N_U3_FB: R42.2, R43.1, U3.4 (VFB)
- new net N_U3_SW: C34.2, L4.1, U3.2 (SW)
- new net N_U3_VBST: C34.1, U3.6 (VBST)
- new net VBUS_DBG: D17.2 (A)
- new net VMON_12V: R45.2, R46.1
- new net VMON_1V8: R49.2, R50.1
- new net VMON_3V3: R47.2, R48.1
- no-connect marks 0 -> 2
Other:
- note added: "Task 5 (power_rails): +12V arrives via global label from power_input, is tapped by U13 IN+ then run through a 2mu03a9 shunt to the internal node +12V_BUCK that feeds U3.VIN. netchecks.txt amends the briefu2019s literal U3.pinfn:VIN=+12V line to +12V_BUCK -- an INA226 truly in series necessarily splits the net (same reasoning as +3V3/+3V3_MOD across U14), and merging both shunt terminals under one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"
