File: sheets/power_rails.kicad_sch (KiCad schematic)
At the start: 31 parts, among them U13 INA226AIDGSR, U14 INA226AIDGSR, U17 AP2112K-3.3TRG1, U3 TPS565201DDCR, U5 AP2112K-1.8TRG1

Commit message: sch: audit fixes — buck EN divider corners, 3V3-domain senses, spec §10 LEDs
F1 (critical): TPS565201 BUCK_EN divider (R40/R41) redesigned against the
datasheet's VENH/VENL/REN corners so the 3.3V buck actually starts once the
12V node is negotiated, without false-starting on pre-negotiation 5V VBUS.

F2 (medium): GP18/GP19 retargeted from the RP2040 sheet to the ethernet
sheet's existing 3.3V-domain PERST/CLKREQ shifter outputs; GP17 gets a new
BSS138 level-shift stage (Q40/R122) on m2, mirroring the Task 10 pattern.

F3 (minor): added the two spec §10 indicator LEDs (D29 12V/power, D30
PD-good) that were dropped during Task 4 and never restored.

check_nets.py all pass; ERC 0 errors / 800 warnings (was 788, full delta
accounted in docs/erc-waivers.md); netlist exports clean, no annotation
warnings.

Co-Authored-By: Claude Fable 5 <noreply@anthropic.com>
Parts:
- R40: value 1.00M -> 36.5k
- R41: value 100k -> 9.31k
Other:
- note added: "Task 13 audit fix (F1, CRITICAL): the original R40=1.00M/R41=100k BUCK_EN divider could never reach TPS565201's VENH (datasheet SLVSE71 Sept-2017 S6.5: VENH min=1.6V, VENL max=0.8V, REN(EN pin pulldown)=120-400k min/typ/max) -- worst case VEN(12V)=0.66-0.90V, always below VENL, buck permanently disabled. A plain 2-resistor divider CANNOT hold VEN below VENL at 5.5V (pre-negotiation VBUS margin) w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"
Changed lines of the file:
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@@
 		(fields_autoplaced yes)
 		(property "Reference" "R40" (at 97 27 0) (effects (font (size 1.27 1.27))))
-		(property "Value" "1.00M" (at 97 33 0) (effects (font (size 1.27 1.27))))
+		(property "Value" "36.5k" (at 97 33 0) (effects (font (size 1.27 1.27))))
 		(property "Footprint" "R_0603" (at 95 30 0) (hide yes) (effects (font (size 1.27 1.27))))
 		(property "Datasheet" "" (at 95 30 0) (hide yes) (effects (font (size 1.27 1.27))))
@@
 		(fields_autoplaced yes)
 		(property "Reference" "R41" (at 97 42 0) (effects (font (size 1.27 1.27))))
-		(property "Value" "100k" (at 97 48 0) (effects (font (size 1.27 1.27))))
+		(property "Value" "9.31k" (at 97 48 0) (effects (font (size 1.27 1.27))))
 		(property "Footprint" "R_0603" (at 95 45 0) (hide yes) (effects (font (size 1.27 1.27))))
 		(property "Datasheet" "" (at 95 45 0) (hide yes) (effects (font (size 1.27 1.27))))
@@
 		(effects (font (size 1.27 1.27)) (justify left bottom))
 	)
+		(text "Task 13 audit fix (F1, CRITICAL): the original R40=1.00M/R41=100k BUCK_EN divider could never reach TPS565201's VENH (datasheet SLVSE71 Sept-2017 S6.5: VENH min=1.6V, VENL max=0.8V, REN(EN pin pulldown)=120-400k min/typ/max) -- worst case VEN(12V)=0.66-0.90V, always below VENL, buck permanently disabled. A plain 2-resistor divider CANNOT hold VEN below VENL at 5.5V (pre-negotiation VBUS margin) while also clearing VENH+10% at 11V (post-negotiation floor) simultaneously -- proven by exhaustive E96 search (0 solutions) and algebraically (required gain VENH/VENL=2.00x exactly equals the 11V/5.5V=2.00x Vin ratio, leaving zero margin for both corners at once). Resolution: EN is the hysteretic UVLO comparator TI's own datasheet graphs name it (S6.6 Fig.3/4 EN Pin UVLO Low/High Voltage) -- the 12V node ramps monotonically from 0V through both test points, so only VENH (the rising threshold) gates turn-on; VENL only matters for a falling edge, which never occurs during power-up. Redesigned R40=36.5k (+12V side, E96), R41=9.31k (GND side, E96) so REN barely perturbs the divider. Four corners (worst-case REN each way): VEN(11V,REN=120k)=2.105V (+31.6% over VENH) -- reliable start; VEN(5.5V,REN=400k)=1.097V (-31.4% under VENH; separately it is above the datasheet's VENL=0.8V but never having crossed VENH on the way up, so per UVLO-latch behavior the buck stays off) -- no false start pre-negotiation. Worst-case actual turn-on crossover (REN=120k, VEN=VENH exactly): Vin=8.36V, matching spec's ~7-8V target closely. Full arithmetic in task-13-report.md Fix pass."
+			(exclude_from_sim no)
+			(at 20 235 0)
+			(effects (font (size 1.27 1.27)) (justify left bottom))
+		)
 	(sheet_instances
 		(path "/"

Commit message: sch: footprints + assembly-split BOM fields
Task 14: bind real footprints to all 363 BOM symbols, add Assembly/LCSC/MPN/
Distributor properties to every symbol, and close the accumulated
footprint_link_issues ERC deferral (148 -> 0).

- New fp-lib-table + lib/sierra-to-usb.pretty/ (15 custom footprints
  authored from real manufacturer drawings: magjack, MHF4, SMA edge,
  nano-SIM, MFF2 eSIM, M.2 socket, bridge rectifier, 2x PoE flyback
  inductors, TPS23730 VQFN-45, FDMC2523P, FOD817 gull-wing DIP-4, SK6805
  LED, PoE transformer, and a corrected full-24-pin USB-C receptacle for
  J1 -- the previously-bound stock footprint only exposed 6 of 24 pins).
- Fixed ~120 bare/stale/wrong-library-prefix Footprint strings project-wide.
- Assembly split: 12 JLC rows (all LCSC-backed), 351 HAND rows (MPN +
  Distributor on every one). Disclosed flip: U30 (eSIM) JLC->HAND per
  sourcing.md's own no-LCSC-listing flag, overriding the task's shorthand.
- Carry-forwards closed: D30 series R 1k->560R, INA226 MSOP-10->VSSOP-10
  (+EP-VIA), R39/R44 Kelvin-route note, JP1-3 solder-jumper footprints,
  SW2 silk note, 42x 0402->0603 hand-solder upgrades.
- New tools/check_footprints.py gate: Footprint/Assembly presence, JLC=>LCSC,
  and footprint-pad-count >= symbol-pin-count (parsed from real .kicad_mod
  files + netlist pin lists).
- Recovered sheets/mcu.kicad_sch from a pre-existing uncommitted data-loss
  state (44 symbols missing vs the Task 13 gate-approved commit) before
  applying any Task 14 edits.

Verification: check_footprints.py all-pass, check_nets.py all-pass
(connectivity untouched), kicad-cli sch erc 0 errors.

Two pre-existing issues disclosed but not fixed here (out of footprint-
assignment scope, documented in docs/verification.md and
docs/erc-waivers.md): J1's now-corrected footprint was masking a Task-7
error, and 7 refs (Q20,Q22-25,Q30,Q31) use letter-pinned generic FET/BJT
symbols that will show unmatched pins at PCB import regardless of
footprint choice -- flagge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
Parts:
- C33, C39: footprint C_0603 -> Capacitor_SMD:C_0603_1608Metric; Assembly (none) -> HAND; Distributor (none) -> LCSC; MPN (none) -> Generic MLCC 0.1uF/16V 0603 (Yageo/Murata/Samsung equiv, ex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
- C34: footprint C_0603 -> Capacitor_SMD:C_0603_1608Metric; Assembly (none) -> HAND; Distributor (none) -> LCSC; MPN (none) -> Generic MLCC 0.1uF/25V 0603 (Yageo/Murata/Samsung equiv, ex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
- C35, C36: footprint C_1210 -> Capacitor_SMD:C_1210_3225Metric; Assembly (none) -> HAND; Distributor (none) -> LCSC; MPN (none) -> Generic MLCC 10uF/25V 1210 (Yageo/Murata/Samsung equiv, exa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
- C37, C38: footprint C_1210 -> Capacitor_SMD:C_1210_3225Metric; Assembly (none) -> HAND; Distributor (none) -> LCSC; MPN (none) -> Generic MLCC 22uF/16V 1210 (Yageo/Murata/Samsung equiv, exa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
- C40, C41, C42, C43: footprint C_0603 -> Capacitor_SMD:C_0603_1608Metric; Assembly (none) -> HAND; Distributor (none) -> LCSC; MPN (none) -> Generic MLCC 1uF/16V 0603 (Yageo/Murata/Samsung equiv, exac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
- D17, D18: footprint D_SOD-323 -> Diode_SMD:D_SOD-323; Assembly (none) -> HAND; Distributor (none) -> LCSC; MPN (none) -> ON Semi B5819W
- L4: footprint L_8x8mm_H4mm -> Inductor_SMD:L_Bourns-SRN8040_8x8.15mm; Assembly (none) -> HAND; Distributor (none) -> LCSC; LCSC (none) -> C36415; MPN (none) -> Sunlord SWPA8040S2R2MT
- R39, R44: footprint R_1206 -> Resistor_SMD:R_1206_3216Metric; Assembly (none) -> HAND; Distributor (none) -> LCSC; KELVIN-ROUTE (none) -> yes; MPN (none) -> Generic 2mOhm 1W 1206 current-sense resistor (order-time eq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
- R40: footprint R_0603 -> Resistor_SMD:R_0603_1608Metric; Assembly (none) -> HAND; Distributor (none) -> LCSC; MPN (none) -> Yageo RC0603JR-0736K5L
- R41: footprint R_0603 -> Resistor_SMD:R_0603_1608Metric; Assembly (none) -> HAND; Distributor (none) -> LCSC; MPN (none) -> Yageo RC0603JR-079K31L
- R42: footprint R_0603 -> Resistor_SMD:R_0603_1608Metric; Assembly (none) -> HAND; Distributor (none) -> LCSC; MPN (none) -> Yageo RC0603JR-0733K2L
- R43, R46: footprint R_0603 -> Resistor_SMD:R_0603_1608Metric; Assembly (none) -> HAND; Distributor (none) -> LCSC; MPN (none) -> Yageo RC0603JR-0710KL
- R45, R47, R48, R49, R50: footprint R_0603 -> Resistor_SMD:R_0603_1608Metric; Assembly (none) -> HAND; Distributor (none) -> LCSC; MPN (none) -> Yageo RC0603JR-07100KL
- U13, U14: footprint Package_SO:MSOP-10_3x3mm_P0.5mm -> Package_SO:HVSSOP-10-1EP_3x3mm_P0.5mm_EP1.83x1.89mm; Assembly (none) -> HAND; Distributor (none) -> LCSC; EP-VIA (none) -> yes; LCSC (none) -> C49851; MPN (none) -> TI INA226AIDGSR
- U17: Assembly (none) -> HAND; Distributor (none) -> LCSC; LCSC (none) -> C51118; MPN (none) -> Diodes AP2112K-3.3TRG1
- U3: Assembly (none) -> HAND; Distributor (none) -> LCSC; LCSC (none) -> C327676; MPN (none) -> TI TPS565201DDCR
- U5: Assembly (none) -> HAND; Distributor (none) -> LCSC; LCSC (none) -> C176944; MPN (none) -> Diodes AP2112K-1.8TRG1

Commit message: sch: resolve all footprint-pad/symbol-pin mismatches from GUI import log
Q20/Q22/Q23: stacked hidden S pins (2,3) added to Q_NMOS_TDSON_PQFN,
matching KiCad's own stock Q_NMOS_SSSGD_AvalancheRated convention, so
TDSON-8-1/PQFN-8-EP's separately-numbered source pads all bind.

U22 (TL431 SOT-23-5): verified against TI's real datasheet (SLVS543S) --
the existing pin binding (K=3/REF=4/A=5) was already correct; pads 1/2 are
datasheet-documented NC/substrate pins, allowlisted rather than rewired.

U13/U14 (INA226): swapped the wrong EP-bearing HVSSOP-10 footprint for the
real no-EP VSSOP-10/MSOP-10 JEDEC MO-187 footprint per TI's SBOS547B
mechanical drawing; removed the now-incorrect EP-VIA property.

J5 (Qwiic JST-SH): switched to KiCad's stock Conn_01x04_MountingPin symbol
pairing convention, added a passive un-grounded MP pin + no-connect flag.

tools/check_footprints.py: added the reverse pad-to-pin coverage check
(catches all of the above) with a documented, datasheet-cited allowlist
for the 3 legitimately-unmapped pads (U22 x2, U30 x1) and stale-entry
detection.

Verification: check_nets.py and check_footprints.py (extended) both pass;
ERC 0 errors / 652 warnings (identical category breakdown to Task-14
baseline); netlist export clean, 363 components / 334 nets unchanged;
net-to-electrode mapping proof table in task-15-report.md confirms zero
connectivity changes beyond the explicitly-authorized additions.

Co-Authored-By: Claude Fable 5 <noreply@anthropic.com>
Parts:
- U13, U14: footprint Package_SO:HVSSOP-10-1EP_3x3mm_P0.5mm_EP1.83x1.89mm -> Package_SO:MSOP-10_3x3mm_P0.5mm; EP-VIA yes -> (none)
Changed lines of the file:
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@@
 		(property "Reference" "U13" (at 47 37 0) (effects (font (size 1.27 1.27))))
 		(property "Value" "INA226AIDGSR" (at 47 43 0) (effects (font (size 1.27 1.27))))
-		(property "Footprint" "Package_SO:HVSSOP-10-1EP_3x3mm_P0.5mm_EP1.83x1.89mm" (at 45 40 0) (hide yes) (effects (font (size 1.27 1.27))))
+		(property "Footprint" "Package_SO:MSOP-10_3x3mm_P0.5mm" (at 45 40 0) (hide yes) (effects (font (size 1.27 1.27))))
 		(property "Datasheet" "" (at 45 40 0) (hide yes) (effects (font (size 1.27 1.27))))
 		(property "Assembly" "HAND" (at 45 40 0) (hide yes) (effects (font (size 1.27 1.27))))
@@
 		(property "MPN" "TI INA226AIDGSR" (at 45 40 0) (hide yes) (effects (font (size 1.27 1.27))))
 		(property "Distributor" "LCSC" (at 45 40 0) (hide yes) (effects (font (size 1.27 1.27))))
-		(property "EP-VIA" "yes" (at 45 40 0) (hide yes) (effects (font (size 1.27 1.27))))
 		(pin "1"
 		)
@@
 		(property "Reference" "U14" (at 197 37 0) (effects (font (size 1.27 1.27))))
 		(property "Value" "INA226AIDGSR" (at 197 43 0) (effects (font (size 1.27 1.27))))
-		(property "Footprint" "Package_SO:HVSSOP-10-1EP_3x3mm_P0.5mm_EP1.83x1.89mm" (at 195 40 0) (hide yes) (effects (font (size 1.27 1.27))))
+		(property "Footprint" "Package_SO:MSOP-10_3x3mm_P0.5mm" (at 195 40 0) (hide yes) (effects (font (size 1.27 1.27))))
 		(property "Datasheet" "" (at 195 40 0) (hide yes) (effects (font (size 1.27 1.27))))
 		(property "Assembly" "HAND" (at 195 40 0) (hide yes) (effects (font (size 1.27 1.27))))
@@
 		(property "MPN" "TI INA226AIDGSR" (at 195 40 0) (hide yes) (effects (font (size 1.27 1.27))))
 		(property "Distributor" "LCSC" (at 195 40 0) (hide yes) (effects (font (size 1.27 1.27))))
-		(property "EP-VIA" "yes" (at 195 40 0) (hide yes) (effects (font (size 1.27 1.27))))
-		(pin "1"
-		)
+		(pin "1"
+		)
