File: sheets/m2.kicad_sch (KiCad schematic)
At the start: 0 parts

Commit message: sch: M.2 socket, vendor-safe VCC policy, strap plane
Task 6: sheets/m2.kicad_sch wired from scratch — CN1 (stock
Connector:Bus_M.2_Socket_B, verified pin-for-pin against verification.md
and the brief before use, no vendor-symbol correction needed), the full
67-pin accounting (GND/VCC/jumpered-VCC/straps/data-plane labels/NC), the
safety-critical strap plane (PCIE_DIS pull-up to +1V8 ONLY per Global
Constraints, VBUS_SENSE divider + force-FET, FCPO_N/W_DISABLE1_N/
MODEM_RESET_N/PERST_N/CLKREQ_N/PEWAKE_N/WAKE_N pull-ups, Q1-Q5 gates with
100k pulldowns for blank-MCU-safe defaults), bulk/decoupling caps, JP1-3
solder jumpers (default open), 9 test points, and the WWAN status LED on
LED_RET. netchecks.txt gets the brief's Step-1 safety assertions (captured
RED against the empty scaffold, now GREEN) and Step-4 data-plane assertions.
ERC 0 errors / 464 warnings (all pre-existing categories, waivers recorded
in docs/erc-waivers.md, including a root-caused lib_symbols-cache bug that
briefly masked the PWR_FLAG forward-reference fix as still broken).

Co-Authored-By: Claude Fable 5 <noreply@anthropic.com>
Parts:
- added C44, C45, C46: 470uF, CP_Elec_6.3x7.7, symbol Device:C_Polarized_Small
- added C47, C48, C49, C50, C51, C52: 10uF, C_0805_2012Metric, symbol Device:C_Small
- added C53, C54, C55, C56, C57: 0.1uF, C_0402_1005Metric, symbol Device:C_Small
- added CN1: EM92xx / RM520N M.2 Key-B (67-pin), Connector_M.2:M.2_Key-B-SMD, symbol Connector:Bus_M.2_Socket_B
- added D19: LED_WWAN_STATUS, LED_SMD:LED_0603_1608Metric, symbol Device:LED
- added JP1, JP2, JP3: SolderJumper_2_Open, Jumper:SolderJumper-2_P1.3mm_Open_Circle, symbol Jumper:SolderJumper_2_Open
- added Q1, Q2, Q3, Q4, Q5: 2N7002, Package_TO_SOT_SMD:SOT-23, symbol Transistor_FET:2N7002
- added R51, R52, R54, R56, R58, R62, R63: 100k, Resistor_SMD:R_0603_1608Metric, symbol Device:R_Small
- added R53, R55, R57, R64, R65, R66: 10k, Resistor_SMD:R_0603_1608Metric, symbol Device:R_Small
- added R59: 33k, Resistor_SMD:R_0603_1608Metric, symbol Device:R_Small
- added R60: 18k, Resistor_SMD:R_0603_1608Metric, symbol Device:R_Small
- added R61, R67: 1k, Resistor_SMD:R_0603_1608Metric, symbol Device:R_Small
- added TP1: FCPO_N, TestPoint:TestPoint_Pad_D1.5mm, symbol Connector:TestPoint
- added TP2: PCIE_DIS, TestPoint:TestPoint_Pad_D1.5mm, symbol Connector:TestPoint
- added TP3: W_DISABLE1_N, TestPoint:TestPoint_Pad_D1.5mm, symbol Connector:TestPoint
- added TP4: MODEM_RESET_N, TestPoint:TestPoint_Pad_D1.5mm, symbol Connector:TestPoint
- added TP5: VBUS_SENSE, TestPoint:TestPoint_Pad_D1.5mm, symbol Connector:TestPoint
- added TP6: WAKE_N, TestPoint:TestPoint_Pad_D1.5mm, symbol Connector:TestPoint
- added TP7: PERST_N, TestPoint:TestPoint_Pad_D1.5mm, symbol Connector:TestPoint
- added TP8: CLKREQ_N, TestPoint:TestPoint_Pad_D1.5mm, symbol Connector:TestPoint
- added TP9: PEWAKE_N, TestPoint:TestPoint_Pad_D1.5mm, symbol Connector:TestPoint
Connections:
- new net +1V8: R53.1, R55.1, R57.1, R61.1, R63.1, R64.1, R65.1, R66.1
- new net +3V3: R51.1, R67.1
- new net +3V3_MOD: C44.1, C45.1, C46.1, C47.1, C48.1, C49.1, C50.1, C51.1, C52.1, C53.1, C54.1, C55.1, C56.1, C57.1, CN1.2 (3.3V), CN1.4 (3.3V), CN1.70 (3.3V), CN1.72 (3.3V), CN1.74 (3.3V), JP1.2 (B), JP2.2 (B), JP3.2 (B)
- new net CLKREQ_N: CN1.52 (~{CLKREQ}), R65.2, TP8.1
- new net FCPO_CTL: Q1.1 (G), R52.1
- new net FCPO_N: CN1.6 (~{FULL_CARD_POWER_OFF}), Q1.3 (D), R51.2, TP1.1
- new net GND: C44.2, C45.2, C46.2, C47.2, C48.2, C49.2, C50.2, C51.2, C52.2, C53.2, C54.2, C55.2, C56.2, C57.2, CN1.11 (GND), CN1.27 (GND), CN1.3 (GND), CN1.33 (GND), CN1.39 (GND), CN1.45 (GND), CN1.5 (GND), CN1.51 (GND), CN1.57 (GND), CN1.71 (GND), CN1.73 (GND), Q1.2 (S), Q2.2 (S), Q3.2 (S), Q4.2 (S), R52.2, R54.2, R56.2, R58.2, R60.2, R62.2
- new net LED_RET: D19.1 (K)
- new net M2_VCC_JP1: CN1.24 (GPIO_7), JP1.1 (A)
- new net M2_VCC_JP2: CN1.38 (DEVSLP), JP2.1 (A)
- new net M2_VCC_JP3: CN1.68 (SUSCLK), JP3.1 (A)
- new net MODEM_RESET_N: CN1.67 (~{RESET}), Q4.3 (D), R57.2, TP4.1
- new net MRST_CTL: Q4.1 (G), R58.1
- new net N_LED_A: D19.2 (A), R67.2
- new net N_Q5_D: Q5.3 (D), R61.2
- new net PCIE_DIS: CN1.20 (GPIO_5), Q2.3 (D), R53.2, TP2.1
- new net PCIE_DIS_CTL: Q2.1 (G), R54.1
- new net PCIE_MRX_N: CN1.47 (PETn0/SATA-A-)
- new net PCIE_MRX_P: CN1.49 (PETp0/SATA-A+)
- new net PCIE_MTX_N: CN1.41 (PERn0/SATA-B+)
- new net PCIE_MTX_P: CN1.43 (PERp0/SATA-B-)
- new net PCIE_REFCLK_N: CN1.53 (REFCLKn)
- new net PCIE_REFCLK_P: CN1.55 (REFCLKp)
- new net PERST_N: CN1.50 (~{PERST}), R64.2, TP7.1
- new net PEWAKE_N: CN1.54 (~{PEWAKE}), R66.2, TP9.1
- new net SS_MOD_RX_N: CN1.29 (PERn1/USB3.0-Rx-/SSIC-RxN)
- new net SS_MOD_RX_P: CN1.31 (PERp1/USB3.0-Rx+/SSIC-RxP)
- new net SS_MOD_TX_C_N: CN1.35 (PETn1/USB3.0-Tx-/SSIC-TxN)
- new net SS_MOD_TX_C_P: CN1.37 (PETp1/USB3.0-Tx+/SSIC-TxP)
- new net UIM1_CLK: CN1.32 (UIM-CLK)
- new net UIM1_DET: CN1.66 (SIM_DETECT)
- new net UIM1_IO: CN1.34 (UIM-DATA)
- new net UIM1_RST: CN1.30 (UIM-RESET)
- new net UIM1_VDD: CN1.36 (UIM-PWR)
- new net UIM2_CLK: CN1.44 (GPIO_2)
- new net UIM2_DET: CN1.40 (GPIO_0)
- new net UIM2_IO: CN1.42 (GPIO_1)
- new net UIM2_RST: CN1.46 (GPIO_3)
- new net UIM2_VDD: CN1.48 (GPIO_4)
- new net USB2_MOD_DM: CN1.9 (USB_D-)
- new net USB2_MOD_DP: CN1.7 (USB_D+)
- new net VBUSSNS_CTL: Q5.1 (G), R62.1
- new net VBUS_DATA: R59.1
- new net VBUS_SENSE: CN1.22 (GPIO_6), Q5.2 (S), R59.2, R60.1, TP5.1
- new net WAKE_N: CN1.23 (GPIO_11), R63.2, TP6.1
- new net WDIS_CTL: Q3.1 (G), R56.1
- new net WWAN_LED_N: CN1.10 (GPIO_9/DAS/~{DSS}/~{LED1})
- new net W_DISABLE1_N: CN1.8 (~{W_DISABLE1}), Q3.3 (D), R55.2, TP3.1
- no-connect marks 0 -> 16
