File: sheets/m2.kicad_sch (KiCad schematic)
At the start: 54 parts, among them CN1 EM92xx / RM520N M.2 Key-B (67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, Q1 2N7002, Q2 2N7002, Q3 2N7002, Q32 DMG3415U-7, Q4 2N7002, Q40 BSS138, Q5 2N7002

Commit message: sch: Task 14 fixes — MPN/footprint agreement, numeric Q pins, durable approximation flags
Parts:
- C53, C54, C55, C56, C57: MPN Generic MLCC 0.1uF 0402 (Yageo/Murata/Samsung equiv, exact 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 -> Generic MLCC 0.1uF X7R 0603 (Yageo/Murata/Samsung equiv, ex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
Changed lines of the file:
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@@
 		(property "Datasheet" "" (at 275 247 0) (hide yes) (effects (font (size 1.27 1.27))))
 		(property "Assembly" "HAND" (at 275 247 0) (hide yes) (effects (font (size 1.27 1.27))))
-		(property "MPN" "Generic MLCC 0.1uF 0402 (Yageo/Murata/Samsung equiv, exact P/N TBD at order)" (at 275 247 0) (hide yes) (effects (font (size 1.27 1.27))))
+		(property "MPN" "Generic MLCC 0.1uF X7R 0603 (Yageo/Murata/Samsung equiv, exact P/N TBD at order)" (at 275 247 0) (hide yes) (effects (font (size 1.27 1.27))))
 		(property "Distributor" "LCSC" (at 275 247 0) (hide yes) (effects (font (size 1.27 1.27))))
 		(pin "1"
@@
 		(property "Datasheet" "" (at 275 256 0) (hide yes) (effects (font (size 1.27 1.27))))
 		(property "Assembly" "HAND" (at 275 256 0) (hide yes) (effects (font (size 1.27 1.27))))
-		(property "MPN" "Generic MLCC 0.1uF 0402 (Yageo/Murata/Samsung equiv, exact P/N TBD at order)" (at 275 256 0) (hide yes) (effects (font (size 1.27 1.27))))
+		(property "MPN" "Generic MLCC 0.1uF X7R 0603 (Yageo/Murata/Samsung equiv, exact P/N TBD at order)" (at 275 256 0) (hide yes) (effects (font (size 1.27 1.27))))
 		(property "Distributor" "LCSC" (at 275 256 0) (hide yes) (effects (font (size 1.27 1.27))))
 		(pin "1"
@@
 		(property "Datasheet" "" (at 275 265 0) (hide yes) (effects (font (size 1.27 1.27))))
 		(property "Assembly" "HAND" (at 275 265 0) (hide yes) (effects (font (size 1.27 1.27))))
-		(property "MPN" "Generic MLCC 0.1uF 0402 (Yageo/Murata/Samsung equiv, exact P/N TBD at order)" (at 275 265 0) (hide yes) (effects (font (size 1.27 1.27))))
+		(property "MPN" "Generic MLCC 0.1uF X7R 0603 (Yageo/Murata/Samsung equiv, exact P/N TBD at order)" (at 275 265 0) (hide yes) (effects (font (size 1.27 1.27))))
 		(property "Distributor" "LCSC" (at 275 265 0) (hide yes) (effects (font (size 1.27 1.27))))
 		(pin "1"
@@
 		(property "Datasheet" "" (at 275 274 0) (hide yes) (effects (font (size 1.27 1.27))))
 		(property "Assembly" "HAND" (at 275 274 0) (hide yes) (effects (font (size 1.27 1.27))))
-		(property "MPN" "Generic MLCC 0.1uF 0402 (Yageo/Murata/Samsung equiv, exact P/N TBD at order)" (at 275 274 0) (hide yes) (effects (font (size 1.27 1.27))))
+		(property "MPN" "Generic MLCC 0.1uF X7R 0603 (Yageo/Murata/Samsung equiv, exact P/N TBD at order)" (at 275 274 0) (hide yes) (effects (font (size 1.27 1.27))))
 		(property "Distributor" "LCSC" (at 275 274 0) (hide yes) (effects (font (size 1.27 1.27))))
 		(pin "1"
@@
 		(property "Datasheet" "" (at 275 283 0) (hide yes) (effects (font (size 1.27 1.27))))
 		(property "Assembly" "HAND" (at 275 283 0) (hide yes) (effects (font (size 1.27 1.27))))
-		(property "MPN" "Generic MLCC 0.1uF 0402 (Yageo/Murata/Samsung equiv, exact P/N TBD at order)" (at 275 283 0) (hide yes) (effects (font (size 1.27 1.27))))
+		(property "MPN" "Generic MLCC 0.1uF X7R 0603 (Yageo/Murata/Samsung equiv, exact P/N TBD at order)" (at 275 283 0) (hide yes) (effects (font (size 1.27 1.27))))
 		(property "Distributor" "LCSC" (at 275 283 0) (hide yes) (effects (font (size 1.27 1.27))))
 		(pin "1"
