File: sheets/mcu.kicad_sch (KiCad schematic)
At the start: 46 parts, among them J4 SWD, J5 Qwiic, J6 Fan, J7 Spare, Q33 DMG3415U-7, Q34 2N7002, SW1 DIP-4, SW2 LED_KILL, SW3 BOOTSEL, SW4 RUN, U24 RP2040, U25 W25Q128JVS, U26 TMP112AIDRLR, U27 TMP112AIDRLR, U28 SK6805-EC15, Y1 12MHz

Commit message: sch: mcu fixes — XOUT crystal resistor, rail-to-rail LED kill, RGB series R, decoupling
Review pass on sheets/mcu.kicad_sch: swap R76 onto the XOUT side of Y1
(XIN direct, 1k limits drive into the crystal per the RPi RP2040 guide);
rebuild the LED-kill gate network rail-to-rail (Q35 2N7002 + repurposed
R82/R84 pull-ups replace the old resistive-mixing divider that left only
~0.2-0.3V of OFF-state Vgs margin — GP9/LED_EN_CTL is now active-low
kill); insert R92 (330R) between GP14 and U28 DIN with a net split
(RGB_DI/RGB_DIN); add decoupling (C78-C81 100nF at U25/U26/U27/RP2040's
9th supply pin, C82 1uF at VREG_VIN); add a Task-14 SW2 silk note and a
power_input.kicad_sch note on D16's unkillable ~75uA glow.

uv run tools/check_nets.py: all pass (new + all pre-existing lines).
kicad-cli sch erc: 0 errors / 611 warnings (600 baseline +11, all
endpoint_off_grid, no new category — see docs/erc-waivers.md).
Parts:
- removed R83: 1.0k, Resistor_SMD:R_0603_1608Metric, symbol Device:R_Small
- added C78, C79, C80, C81: 100nF, Capacitor_SMD:C_0402_1005Metric, symbol Device:C_Small
- added C82: 1uF, Capacitor_SMD:C_0603_1608Metric, symbol Device:C_Small
- added Q35: 2N7002, Package_TO_SOT_SMD:SOT-23, symbol Transistor_FET:2N7002
- added R92: 330, Resistor_SMD:R_0402_1005Metric, symbol Device:R_Small
- R84: value 10.0k -> 100k
Connections:
- net +3V3: now also R82.2
- net +3V3_MCU: now also R84.2, C78.1, C79.1, C80.1, C81.1, C82.1
- net GND: now also C78.2, C79.2, C80.2, C81.2, C82.2, Q35.2 (S); no longer R82.2
- net LED_EN_CTL: now also R84.1, Q35.1 (G); no longer R84.2
- net N_LEDKILL_GATE: no longer R84.1
- net N_SW2_KILL: now also Q35.3 (D)
- net RGB_DI: now also R92.1; no longer U28.1 (DIN)
- net XTAL_XIN: now also C73.1, Y1.1; no longer R76.1
- net XTAL_XOUT: now also R76.1; no longer C74.1, Y1.3
- removed net XTAL1: C73.1, R76.2, Y1.1
- new net N_XOUT_R: C74.1, R76.2, Y1.3
- new net RGB_DIN: R92.2, U28.1 (DIN)
Other:
- note added: "Decoupling shortfall (review Fix 4): added C78 (100nF, at U25 flash VCC pin), C79 (100nF, at U26 V+ pin), C80 (100nF, at U27 V+ pin) -- none had a dedicated local bypass cap before this fix. Added C81 (100nF) as the 9th RP2040 supply-pin decoupling cap (U24 has 9 +3V3_MCU-referenced supply pins per the RPi "Hardware design with RP2040" guide -- IOVDD x6 + ADC_AVDD + VREG_VIN + USB_VDD; only 8 100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"
- note added: "LED-kill gate logic (rail-to-rail rebuild, review-pass Fix 2): Q33 (DMG3415U-7, P-FET) gate node N_LEDKILL_GATE has a 100k pull-up (R82) to +3V3 (default-OFF contribution) and SW2's common leg. SW2 throw A -> N_SW2_KILL -> Q35 (2N7002) drain; Q35 source=GND; Q35 gate=LED_EN_CTL with a 100k pull-up (R84) to +3V3_MCU -- so blank-MCU/hi-Z GP9 = Q35 ON. SW2 throw C = no-connect (OFF position). Truth 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"
- note added: "RGB_DI series R (review Fix 3): R92 (330R) inserted between GP14 and U28 DIN -- GP14 side stays net RGB_DI, U28.DIN side is net RGB_DIN. Firmware: idle DIN low when LED_PWR killed."
- note added: "Task-14 note: SW2 silk must label ON/KILL positions (review Fix 5c) -- SW2 throw A = ON (LEDs enabled per the rail-to-rail kill network, Fix 2), throw C = KILL/unused-NC side. Silkscreen legend needed so the physical slide position is unambiguous to an assembler/end-user."
- note removed: "LED-kill gate logic (high-side, amendment 1): default (SW2 idle + GP9 released) -> R84 100k pulldown -> gate=0V -> Q33 ON -> LED_PWR=+3V3 (LEDs on). SW2 engaged (throw A) OR GP9 driven HIGH -> gate pulled toward +3V3 through 1k (SW2) or 10k (GP9) -> |Vgs| << DMG3415U-7 threshold -> Q33 OFF -> LEDs dark. R83=1k dominates R84/R85 even if GP9 is simultaneously driven LOW (worst-case conflict still y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"

Commit message: sch: mcu — R84 10k (blank-MCU pull-down fight), GPIO table polarity row
Re-review regression fix: R84 (Q35 gate pull-up to +3V3_MCU) back to 10k
from 100k — RP2040 pads reset with the internal pull-down (~50-80k)
enabled, so 100k divided a blank MCU's LED_EN_CTL to ~1.10-1.47V, inside
the 2N7002's Vgs(th) band (LEDs off/indeterminate instead of the required
blank-MCU-default ON). With 10k: Vgs(Q35) = 3.3*50/60 = 2.75V (worst) to
3.3*80/90 = 2.93V, above the 2.5V worst-case threshold; GP9 LOW still
overrides trivially; no other truth-table row affected. Sheet note,
netchecks comment, and task-9-report.md arithmetic updated; the report's
binding GPIO map row for GP9 corrected to "active-LOW kill / hi-Z=on"
(was still describing the superseded active-HIGH design).

uv run tools/check_nets.py: all pass. ERC: 0 errors / 611 warnings
(unchanged). Netlist export clean; R84 nets verified unchanged.
Parts:
- R84: value 100k -> 10.0k
Other:
- note added: "LED-kill gate logic (rail-to-rail rebuild, review-pass Fix 2): Q33 (DMG3415U-7, P-FET) gate node N_LEDKILL_GATE has a 100k pull-up (R82) to +3V3 (default-OFF contribution) and SW2's common leg. SW2 throw A -> N_SW2_KILL -> Q35 (2N7002) drain; Q35 source=GND; Q35 gate=LED_EN_CTL with a 10k pull-up (R84) to +3V3_MCU -- so blank-MCU/hi-Z GP9 = Q35 ON. R84 is 10k (NOT 100k): RP2040 pads reset with th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"
- note removed: "LED-kill gate logic (rail-to-rail rebuild, review-pass Fix 2): Q33 (DMG3415U-7, P-FET) gate node N_LEDKILL_GATE has a 100k pull-up (R82) to +3V3 (default-OFF contribution) and SW2's common leg. SW2 throw A -> N_SW2_KILL -> Q35 (2N7002) drain; Q35 source=GND; Q35 gate=LED_EN_CTL with a 100k pull-up (R84) to +3V3_MCU -- so blank-MCU/hi-Z GP9 = Q35 ON. SW2 throw C = no-connect (OFF position). Truth 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"
Changed lines of the file:
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@@
 		(fields_autoplaced yes)
 		(property "Reference" "R84" (at 227 172 0) (effects (font (size 1.27 1.27))))
-		(property "Value" "100k" (at 227 178 0) (effects (font (size 1.27 1.27))))
+		(property "Value" "10.0k" (at 227 178 0) (effects (font (size 1.27 1.27))))
 		(property "Footprint" "Resistor_SMD:R_0603_1608Metric" (at 225 175 0) (hide yes) (effects (font (size 1.27 1.27))))
 		(property "Datasheet" "" (at 225 175 0) (hide yes) (effects (font (size 1.27 1.27))))
@@
 		(effects (font (size 1.016 1.016)) (justify left bottom))
 	)
-	(text "LED-kill gate logic (rail-to-rail rebuild, review-pass Fix 2): Q33 (DMG3415U-7, P-FET) gate node N_LEDKILL_GATE has a 100k pull-up (R82) to +3V3 (default-OFF contribution) and SW2's common leg. SW2 throw A -> N_SW2_KILL -> Q35 (2N7002) drain; Q35 source=GND; Q35 gate=LED_EN_CTL with a 100k pull-up (R84) to +3V3_MCU -- so blank-MCU/hi-Z GP9 = Q35 ON. SW2 throw C = no-connect (OFF position).\nTruth table: SW2-ON + GP9 hi-Z/high -> Q35 ON -> N_SW2_KILL~0V -> gate~0V, Vgs=-3.3V -> LEDs ON (blank-MCU default). SW2-OFF -> gate=3.3V via R82 regardless of GP9/Q35 -> Q33 OFF (hardware wins). SW2-ON + GP9 driven LOW -> Q35 OFF -> SW2 branch open -> gate=3.3V via R82 -> Q33 OFF (firmware kill). All three states are rail-to-rail (no resistive-divider margin) -- see task-9-report.md Fix-pass section for arithmetic.\nLED_EN_CTL polarity note: GP9 is now an ACTIVE-LOW kill line (driving LOW forces LEDs off through Q35); hi-Z/floating = LEDs on by default. This is the OPPOSITE polarity of the prior resistive-mixing design's GP9-HIGH-kills convention -- firmware must be updated."
+	(text "LED-kill gate logic (rail-to-rail rebuild, review-pass Fix 2): Q33 (DMG3415U-7, P-FET) gate node N_LEDKILL_GATE has a 100k pull-up (R82) to +3V3 (default-OFF contribution) and SW2's common leg. SW2 throw A -> N_SW2_KILL -> Q35 (2N7002) drain; Q35 source=GND; Q35 gate=LED_EN_CTL with a 10k pull-up (R84) to +3V3_MCU -- so blank-MCU/hi-Z GP9 = Q35 ON. R84 is 10k (NOT 100k): RP2040 pads reset with the internal pull-DOWN enabled (~50-80k), so a 100k pull-up would divide LED_EN_CTL to ~1.10-1.47V, inside the 2N7002's Vgs(th) band; 10k keeps the blank-MCU gate at 3.3*50/60=2.75V to 3.3*80/90=2.93V, above the 2.5V worst-case threshold. SW2 throw C = no-connect (OFF position).\nTruth table: SW2-ON + GP9 hi-Z/high -> Q35 ON -> N_SW2_KILL~0V -> gate~0V, Vgs=-3.3V -> LEDs ON (blank-MCU default). SW2-OFF -> gate=3.3V via R82 regardless of GP9/Q35 -> Q33 OFF (hardware wins). SW2-ON + GP9 driven LOW -> Q35 OFF -> SW2 branch open -> gate=3.3V via R82 -> Q33 OFF (firmware kill). All Q33 gate states are rail-to-rail (no resistive-divider margin) -- see task-9-report.md Fix-pass section for arithmetic.\nLED_EN_CTL polarity note: GP9 is now an ACTIVE-LOW kill line (driving LOW forces LEDs off through Q35); hi-Z/floating = LEDs on by default. This is the OPPOSITE polarity of the prior resistive-mixing design's GP9-HIGH-kills convention -- firmware must be updated."
 		(at 200 195 0)
 		(effects (font (size 1.27 1.27)))
