File: sheets/mcu.kicad_sch (KiCad schematic)
At the start: 52 parts, among them J4 SWD, J5 Qwiic, J6 Fan, J7 Spare, Q33 DMG3415U-7, Q34 2N7002, Q35 2N7002, SW1 DIP-4, SW2 LED_KILL, SW3 BOOTSEL, SW4 RUN, U24 RP2040, U25 W25Q128JVS, U26 TMP112AIDRLR, U27 TMP112AIDRLR, U28 SK6805-EC15, Y1 12MHz

Commit message: sch: audit fixes — buck EN divider corners, 3V3-domain senses, spec §10 LEDs
F1 (critical): TPS565201 BUCK_EN divider (R40/R41) redesigned against the
datasheet's VENH/VENL/REN corners so the 3.3V buck actually starts once the
12V node is negotiated, without false-starting on pre-negotiation 5V VBUS.

F2 (medium): GP18/GP19 retargeted from the RP2040 sheet to the ethernet
sheet's existing 3.3V-domain PERST/CLKREQ shifter outputs; GP17 gets a new
BSS138 level-shift stage (Q40/R122) on m2, mirroring the Task 10 pattern.

F3 (minor): added the two spec §10 indicator LEDs (D29 12V/power, D30
PD-good) that were dropped during Task 4 and never restored.

check_nets.py all pass; ERC 0 errors / 800 warnings (was 788, full delta
accounted in docs/erc-waivers.md); netlist exports clean, no annotation
warnings.

Co-Authored-By: Claude Fable 5 <noreply@anthropic.com>
Connections:
- net CLKREQ_N renamed N_CLKREQ_3V3
- net PERST_N renamed N_PERST_3V3
- net WAKE_N renamed WAKE_3V3
Changed lines of the file:
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@@
 		(property "Intersheetrefs" "${INTERSHEET_REFS}" (at 175.4 102.54 0) (effects (font (size 1.27 1.27))))
 	)
-	(global_label "WAKE_N"
+	(global_label "WAKE_3V3"
 		(shape input)
 		(at 175.4 105.08 0)
@@
 		(property "Intersheetrefs" "${INTERSHEET_REFS}" (at 175.4 105.08 0) (effects (font (size 1.27 1.27))))
 	)
-	(global_label "PERST_N"
+	(global_label "N_PERST_3V3"
 		(shape input)
 		(at 175.4 107.62 0)
@@
 		(property "Intersheetrefs" "${INTERSHEET_REFS}" (at 175.4 107.62 0) (effects (font (size 1.27 1.27))))
 	)
-	(global_label "CLKREQ_N"
+	(global_label "N_CLKREQ_3V3"
 		(shape input)
 		(at 175.4 110.16 0)

Commit message: sch: footprints + assembly-split BOM fields
Task 14: bind real footprints to all 363 BOM symbols, add Assembly/LCSC/MPN/
Distributor properties to every symbol, and close the accumulated
footprint_link_issues ERC deferral (148 -> 0).

- New fp-lib-table + lib/sierra-to-usb.pretty/ (15 custom footprints
  authored from real manufacturer drawings: magjack, MHF4, SMA edge,
  nano-SIM, MFF2 eSIM, M.2 socket, bridge rectifier, 2x PoE flyback
  inductors, TPS23730 VQFN-45, FDMC2523P, FOD817 gull-wing DIP-4, SK6805
  LED, PoE transformer, and a corrected full-24-pin USB-C receptacle for
  J1 -- the previously-bound stock footprint only exposed 6 of 24 pins).
- Fixed ~120 bare/stale/wrong-library-prefix Footprint strings project-wide.
- Assembly split: 12 JLC rows (all LCSC-backed), 351 HAND rows (MPN +
  Distributor on every one). Disclosed flip: U30 (eSIM) JLC->HAND per
  sourcing.md's own no-LCSC-listing flag, overriding the task's shorthand.
- Carry-forwards closed: D30 series R 1k->560R, INA226 MSOP-10->VSSOP-10
  (+EP-VIA), R39/R44 Kelvin-route note, JP1-3 solder-jumper footprints,
  SW2 silk note, 42x 0402->0603 hand-solder upgrades.
- New tools/check_footprints.py gate: Footprint/Assembly presence, JLC=>LCSC,
  and footprint-pad-count >= symbol-pin-count (parsed from real .kicad_mod
  files + netlist pin lists).
- Recovered sheets/mcu.kicad_sch from a pre-existing uncommitted data-loss
  state (44 symbols missing vs the Task 13 gate-approved commit) before
  applying any Task 14 edits.

Verification: check_footprints.py all-pass, check_nets.py all-pass
(connectivity untouched), kicad-cli sch erc 0 errors.

Two pre-existing issues disclosed but not fixed here (out of footprint-
assignment scope, documented in docs/verification.md and
docs/erc-waivers.md): J1's now-corrected footprint was masking a Task-7
error, and 7 refs (Q20,Q22-25,Q30,Q31) use letter-pinned generic FET/BJT
symbols that will show unmatched pins at PCB import regardless of
footprint choice -- flagge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
Parts:
- C65, C66, C67, C68, C69, C70, C72, C75, C76, C77, C78, C79, C80, C81: footprint Capacitor_SMD:C_0402_1005Metric -> Capacitor_SMD:C_0603_1608Metric; Assembly (none) -> HAND; Distributor (none) -> LCSC; MPN (none) -> Generic MLCC 100nF 0402 (Yageo/Murata/Samsung equiv, exact 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
- C71, C82: Assembly (none) -> HAND; Distributor (none) -> LCSC; MPN (none) -> Generic MLCC 1uF 0603 (Yageo/Murata/Samsung equiv, exact P/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
- C73, C74: footprint Capacitor_SMD:C_0402_1005Metric -> Capacitor_SMD:C_0603_1608Metric; Assembly (none) -> HAND; Distributor (none) -> LCSC; MPN (none) -> Generic MLCC 27pF 0402 (Yageo/Murata/Samsung equiv, exact P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
- D26: Assembly (none) -> HAND; Distributor (none) -> LCSC; MPN (none) -> 1N4148W
- J4: Assembly (none) -> HAND; Distributor (none) -> LCSC; MPN (none) -> Generic 2.54mm pin header 1x03
- J5: footprint Connector_JST:JST_SH_SM04B-SRSS-TB_1x04-1MP_P1.00mm -> Connector_JST:JST_SH_SM04B-SRSS-TB_1x04-1MP_P1.00mm_Horizontal; Assembly (none) -> JLC; Distributor (none) -> LCSC; LCSC (none) -> C160390; MPN (none) -> JST BM04B-SRSS-TB(LF)(SN)
- J6: Assembly (none) -> HAND; Distributor (none) -> LCSC; MPN (none) -> Generic 2.54mm pin header 1x02
- J7: Assembly (none) -> HAND; Distributor (none) -> LCSC; MPN (none) -> Generic 2.54mm pin header 1x04
- Q33: Assembly (none) -> HAND; Distributor (none) -> LCSC; LCSC (none) -> C96616; MPN (none) -> Diodes DMG3415U-7
- Q34, Q35: Assembly (none) -> HAND; Distributor (none) -> LCSC; LCSC (none) -> C8545; MPN (none) -> 2N7002
- R76: footprint Resistor_SMD:R_0402_1005Metric -> Resistor_SMD:R_0603_1608Metric; Assembly (none) -> HAND; Distributor (none) -> LCSC; MPN (none) -> Yageo RC0402JR-071KL
- R77: footprint Resistor_SMD:R_0402_1005Metric -> Resistor_SMD:R_0603_1608Metric; Assembly (none) -> HAND; Distributor (none) -> LCSC; MPN (none) -> Yageo RC0402JR-0710KL
- R78, R79: footprint Resistor_SMD:R_0402_1005Metric -> Resistor_SMD:R_0603_1608Metric; Assembly (none) -> HAND; Distributor (none) -> LCSC; MPN (none) -> Yageo RC0402JR-0727R4L
- R80, R81: Assembly (none) -> HAND; Distributor (none) -> LCSC; MPN (none) -> Yageo RC0603JR-074K7L
- R82, R85, R87, R88, R89, R90, R91: Assembly (none) -> HAND; Distributor (none) -> LCSC; MPN (none) -> Yageo RC0603JR-07100KL
- R84: Assembly (none) -> HAND; Distributor (none) -> LCSC; MPN (none) -> Yageo RC0603JR-0710KL
- R86: Assembly (none) -> HAND; Distributor (none) -> LCSC; MPN (none) -> Yageo RC0603JR-0722KL
- R92: footprint Resistor_SMD:R_0402_1005Metric -> Resistor_SMD:R_0603_1608Metric; Assembly (none) -> HAND; Distributor (none) -> LCSC; MPN (none) -> Yageo RC0402JR-07330RL
- SW1: footprint Button_Switch_THT:SW_DIP_x04 -> Button_Switch_THT:SW_DIP_SPSTx04_Piano_10.8x11.72mm_W7.62mm_P2.54mm; Assembly (none) -> HAND; Distributor (none) -> LCSC; LCSC (none) -> C99418; MPN (none) -> DSWB04LHGET
- SW2: footprint Button_Switch_THT:SW_SPDT_PCM12 -> Button_Switch_SMD:SW_SPDT_PCM12; Assembly (none) -> HAND; Distributor (none) -> LCSC; LCSC (none) -> C221841; MPN (none) -> C&K PCM12SMTR; SilkNote (none) -> ON/KILL
- SW3, SW4: Assembly (none) -> HAND; Distributor (none) -> LCSC; MPN (none) -> Omron B3U-1000P
- U24: Assembly (none) -> JLC; Distributor (none) -> LCSC; LCSC (none) -> C2040; MPN (none) -> Raspberry Pi RP2040
- U25: Assembly (none) -> JLC; Distributor (none) -> LCSC; LCSC (none) -> C97521; MPN (none) -> Winbond W25Q128JVSIQ
- U26, U27: Assembly (none) -> HAND; Distributor (none) -> LCSC; LCSC (none) -> C28927; MPN (none) -> TI TMP112AIDRLR
- U28: footprint LED_SMD:LED_SK6805-EC15_1.5x1.5mm -> sierra-to-usb:LED_SK6805-EC15_1.5x1.5mm; Assembly (none) -> HAND; Distributor (none) -> LCSC; LCSC (none) -> C2890035; MPN (none) -> OPSCO SK6805-EC15
- Y1: Assembly (none) -> HAND; Distributor (none) -> LCSC; MPN (none) -> Generic 12MHz (order-time equiv)
