File: sheets/mcu.kicad_sch (KiCad schematic)
At the start: 52 parts, among them J4 SWD, J5 Qwiic, J6 Fan, J7 Spare, Q33 DMG3415U-7, Q34 2N7002, Q35 2N7002, SW1 DIP-4, SW2 LED_KILL, SW3 BOOTSEL, SW4 RUN, U24 RP2040, U25 W25Q128JVS, U26 TMP112AIDRLR, U27 TMP112AIDRLR, U28 SK6805-EC15, Y1 12MHz

Commit message: sch: Task 14 fixes — MPN/footprint agreement, numeric Q pins, durable approximation flags
Parts:
- C65, C66, C67, C68, C69, C70, C72, C75, C76, C77, C78, C79, C80, C81: MPN Generic MLCC 100nF 0402 (Yageo/Murata/Samsung equiv, exact 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 -> Generic MLCC 100nF X7R 0603 (Yageo/Murata/Samsung equiv, ex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
- C73, C74: MPN Generic MLCC 27pF 0402 (Yageo/Murata/Samsung equiv, exact P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 -> Generic MLCC 27pF C0G 0603 (Yageo/Murata/Samsung equiv, exa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
- R76: MPN Yageo RC0402JR-071KL -> Yageo RC0603JR-071KL
- R77: MPN Yageo RC0402JR-0710KL -> Yageo RC0603JR-0710KL
- R78, R79: MPN Yageo RC0402JR-0727R4L -> Yageo RC0603JR-0727R4L
- R92: MPN Yageo RC0402JR-07330RL -> Yageo RC0603JR-07330RL
