File: sheets/ethernet.kicad_sch (KiCad schematic)
At the start: 0 parts

Commit message: sch: RTL8125BG + 2.5G PoE magjack
Parts:
- added C100, C101, C102, C89, C90, C91, C92, C93, C94, C95, C96, C97, C98, C99: 100nF, Capacitor_SMD:C_0402_1005Metric, symbol Device:C_Small
- added C103: 1nF, Capacitor_SMD:C_0603_1608Metric, symbol Device:C_Small
- added C104, C105, C106, C107: 22nF 100V, Capacitor_SMD:C_0603_1608Metric, symbol Device:C_Small
- added C108: 1000pF 2kV, Capacitor_SMD:C_0603_1608Metric, symbol Device:C_Small
- added C83, C84: 220nF, Capacitor_SMD:C_0603_1608Metric, symbol Device:C_Small
- added C85, C86: 27pF, Capacitor_SMD:C_0603_1608Metric, symbol Device:C_Small
- added C87, C88: 1uF, Capacitor_SMD:C_0603_1608Metric, symbol Device:C_Small
- added J8: 2250504-1, symbol sierra-to-usb:Bel2250504-1
- added Q36, Q37, Q38: 2N7002, Package_TO_SOT_SMD:SOT-23, symbol Transistor_FET:2N7002
- added R100, R101, R98, R99: 75, Resistor_SMD:R_0603_1608Metric, symbol Device:R_Small
- added R93, R94, R95: 10k, Resistor_SMD:R_0603_1608Metric, symbol Device:R_Small
- added R96: 2.49k 1%, Resistor_SMD:R_0603_1608Metric, symbol Device:R_Small
- added R97: 4.7k, Resistor_SMD:R_0603_1608Metric, symbol Device:R_Small
- added TP11: LED3, TestPoint:TestPoint_Pad_D1.5mm, symbol Connector:TestPoint
- added U11: 93C46, Package_SO:SOIC-8_3.9x4.9mm_P1.27mm, symbol sierra-to-usb:93C46
- added U12: AP2112K-1.0, Package_TO_SOT_SMD:SOT-23-5, symbol sierra-to-usb:AP2112K-1.0
- added U9: RTL8125BG-CG, Package_DFN_QFN:QFN-48-1EP_6x6mm_P0.4mm_EP4.3x4.3mm, symbol sierra-to-usb:RTL8125BG
- added Y2: 25MHz, Crystal:Crystal_SMD_3225-4Pin_3.2x2.5mm, symbol Device:Crystal_GND24
Connections:
- new net +0V95: C100.1, C101.1, C102.1, C88.1, C96.1, C97.1, C98.1, C99.1, U12.5 (VOUT), U9.11 (AVDD09), U9.16 (AVDD09), U9.22 (AVDD09), U9.28 (DVDD09), U9.37 (EVDD09), U9.47 (DVDD09), U9.8 (DVDD09)
- new net +1V8: Q36.1 (G), Q37.1 (G), Q38.1 (G)
- new net +3V3: C87.1, C89.1, C90.1, C91.1, C92.1, C93.1, C94.1, C95.1, R93.2, R94.2, R95.2, R97.2, U11.6 (ORG), U11.8 (VCC), U12.1 (VIN), U9.15 (AVDD33), U9.19 (AVDD33), U9.29 (DVDD33), U9.33 (AVDD33), U9.34 (AVDD33_XTAL), U9.43 (EVDD33), U9.46 (DVDD33)
- new net CLKREQ_N: Q37.2 (S)
- new net GND: C100.2, C101.2, C102.2, C103.2, C108.2, C85.2, C86.2, C87.2, C88.2, C89.2, C90.2, C91.2, C92.2, C93.2, C94.2, C95.2, C96.2, C97.2, C98.2, C99.2, J8.SH, R96.2, U11.5 (GND), U12.2 (GND), U9.32 (EEPROM_SEL), U9.40 (GND), U9.49 (GND), Y2.2 (G), Y2.4 (G)
- new net LED0: U11.3 (DI), U9.30 (LED0/EEDI)
- new net LED1: R97.1, U11.2 (CLK), U9.27 (LED1/EESK)
- new net LED3: TP11.1, U9.35 (LED3)
- new net MDI0_N: J8.11 (TRD1-), U9.14 (MDIN0)
- new net MDI0_P: J8.10 (TRD1+), U9.13 (MDIP0)
- new net MDI1_N: J8.5 (TRD2-), U9.18 (MDIN1)
- new net MDI1_P: J8.4 (TRD2+), U9.17 (MDIP1)
- new net MDI2_N: J8.2 (TRD3-), U9.21 (MDIN2)
- new net MDI2_P: J8.3 (TRD3+), U9.20 (MDIP2)
- new net MDI3_N: J8.9 (TRD4-), U9.24 (MDIN3)
- new net MDI3_P: J8.8 (TRD4+), U9.23 (MDIP3)
- new net N_BOBSMITH: C104.2, C105.2, C106.2, C107.2, C108.1
- new net N_BS_13: C104.1, R98.2
- new net N_BS_14: C105.1, R99.2
- new net N_BS_15: C106.1, R100.2
- new net N_BS_16: C107.1, R101.2
- new net N_CLKREQ_3V3: Q37.3 (D), R94.1, U9.48 (CLKREQB)
- new net N_EXT095_EN: U12.3 (EN), U9.6 (POW_EXT_SWR)
- new net N_PERST_3V3: Q36.3 (D), R93.1, U9.36 (PERSTB)
- new net N_PEWAKE_3V3: Q38.3 (D), R95.1, U9.2 (LANWAKEB)
- new net N_RSET: R96.1, U9.12 (RSET)
- new net N_TRCT_COMMON: C103.1, J8.1 (TRCT3), J8.12 (TRCT1), J8.6 (TRCT2), J8.7 (TRCT4)
- new net N_XTAL1: C86.1, U9.10 (CKXTAL1), Y2.3
- new net N_XTAL2: C85.1, U9.9 (CKXTAL2), Y2.1
- new net PCIE_MRX_C_N: C84.1, U9.39 (HSON)
- new net PCIE_MRX_C_P: C83.1, U9.38 (HSOP)
- new net PCIE_MRX_N: C84.2
- new net PCIE_MRX_P: C83.2
- new net PCIE_MTX_N: U9.42 (HSIN)
- new net PCIE_MTX_P: U9.41 (HSIP)
- new net PCIE_REFCLK_N: U9.45 (REFCLK_N)
- new net PCIE_REFCLK_P: U9.44 (REFCLK_P)
- new net PERST_N: Q36.2 (S)
- new net PEWAKE_N: Q38.2 (S)
- new net POE_VA+: J8.13 (VC12), R98.1
- new net POE_VA-: J8.14 (VC36), R99.1
- new net POE_VB+: J8.15 (VC45), R100.1
- new net POE_VB-: J8.16 (VC78), R101.1
- new net RTL_EE_CS: U11.1 (CS), U9.31 (EECS)
- new net RTL_EE_DO: U11.4 (DO), U9.25 (LED2/EEDO)
- new net RTL_RST_N: U9.1 (ISOLATEB)
- no-connect marks 0 -> 6
