File: sheets/ethernet.kicad_sch (KiCad schematic)
At the start: 58 parts, among them J8 2250504-1, Q36 BSS138, Q37 BSS138, Q38 BSS138, U11 93C46, U12 TLV62569DBVR, U15 TPS62933FDRLR, U9 RTL8125BG-CG, Y2 25MHz

Commit message: sch: footprints + assembly-split BOM fields
Task 14: bind real footprints to all 363 BOM symbols, add Assembly/LCSC/MPN/
Distributor properties to every symbol, and close the accumulated
footprint_link_issues ERC deferral (148 -> 0).

- New fp-lib-table + lib/sierra-to-usb.pretty/ (15 custom footprints
  authored from real manufacturer drawings: magjack, MHF4, SMA edge,
  nano-SIM, MFF2 eSIM, M.2 socket, bridge rectifier, 2x PoE flyback
  inductors, TPS23730 VQFN-45, FDMC2523P, FOD817 gull-wing DIP-4, SK6805
  LED, PoE transformer, and a corrected full-24-pin USB-C receptacle for
  J1 -- the previously-bound stock footprint only exposed 6 of 24 pins).
- Fixed ~120 bare/stale/wrong-library-prefix Footprint strings project-wide.
- Assembly split: 12 JLC rows (all LCSC-backed), 351 HAND rows (MPN +
  Distributor on every one). Disclosed flip: U30 (eSIM) JLC->HAND per
  sourcing.md's own no-LCSC-listing flag, overriding the task's shorthand.
- Carry-forwards closed: D30 series R 1k->560R, INA226 MSOP-10->VSSOP-10
  (+EP-VIA), R39/R44 Kelvin-route note, JP1-3 solder-jumper footprints,
  SW2 silk note, 42x 0402->0603 hand-solder upgrades.
- New tools/check_footprints.py gate: Footprint/Assembly presence, JLC=>LCSC,
  and footprint-pad-count >= symbol-pin-count (parsed from real .kicad_mod
  files + netlist pin lists).
- Recovered sheets/mcu.kicad_sch from a pre-existing uncommitted data-loss
  state (44 symbols missing vs the Task 13 gate-approved commit) before
  applying any Task 14 edits.

Verification: check_footprints.py all-pass, check_nets.py all-pass
(connectivity untouched), kicad-cli sch erc 0 errors.

Two pre-existing issues disclosed but not fixed here (out of footprint-
assignment scope, documented in docs/verification.md and
docs/erc-waivers.md): J1's now-corrected footprint was masking a Task-7
error, and 7 refs (Q20,Q22-25,Q30,Q31) use letter-pinned generic FET/BJT
symbols that will show unmatched pins at PCB import regardless of
footprint choice -- flagge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
Parts:
- C100, C110, C87, C88, C99: Assembly (none) -> HAND; Distributor (none) -> LCSC; MPN (none) -> Generic MLCC 10uF 0603 (Yageo/Murata/Samsung equiv, exact P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
- C101, C90, C91, C95, C96, C97, C98: Assembly (none) -> HAND; Distributor (none) -> LCSC; MPN (none) -> Generic MLCC 2.2uF 0603 (Yageo/Murata/Samsung equiv, exact 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
- C102, C94: Assembly (none) -> HAND; Distributor (none) -> LCSC; MPN (none) -> Generic MLCC 1uF 0603 (Yageo/Murata/Samsung equiv, exact P/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
- C103: Assembly (none) -> HAND; Distributor (none) -> LCSC; MPN (none) -> Generic MLCC 390pF 0603 (Yageo/Murata/Samsung equiv, exact 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
- C109: Assembly (none) -> HAND; Distributor (none) -> LCSC; MPN (none) -> Generic MLCC 1nF 0603 (Yageo/Murata/Samsung equiv, exact P/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
- C111, C113, C89, C92, C93: footprint Capacitor_SMD:C_0402_1005Metric -> Capacitor_SMD:C_0603_1608Metric; Assembly (none) -> HAND; Distributor (none) -> LCSC; MPN (none) -> Generic MLCC 100nF 0402 (Yageo/Murata/Samsung equiv, exact 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
- C112: Assembly (none) -> HAND; Distributor (none) -> LCSC; MPN (none) -> Generic MLCC 10nF 0603 (Yageo/Murata/Samsung equiv, exact P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
- C114, C115: Assembly (none) -> HAND; Distributor (none) -> LCSC; MPN (none) -> Generic MLCC 22uF 0805 (Yageo/Murata/Samsung equiv, exact P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
- C83, C84: Assembly (none) -> HAND; Distributor (none) -> LCSC; MPN (none) -> Generic MLCC 220nF 0603 (Yageo/Murata/Samsung equiv, exact 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
- C85, C86: Assembly (none) -> HAND; Distributor (none) -> LCSC; MPN (none) -> Generic MLCC 27pF 0603 (Yageo/Murata/Samsung equiv, exact P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
- D10: Assembly (none) -> HAND; Distributor (none) -> LCSC; MPN (none) -> Generic green 0603 LED (Yageo/Everlight equiv)
- FB1: Assembly (none) -> HAND; Distributor (none) -> LCSC; LCSC (none) -> C88984; MPN (none) -> Murata BLM18PG330SN1D
- J8: footprint (none) -> sierra-to-usb:Bel_2250504-1; Assembly (none) -> HAND; Distributor (none) -> DigiKey; MPN (none) -> Bel 2250504-1
- L5, L6: Assembly (none) -> HAND; Distributor (none) -> LCSC; MPN (none) -> Generic 2.2uH shielded SMD inductor, 1210 (order-time equiv)
- Q36, Q37, Q38: Assembly (none) -> HAND; Distributor (none) -> LCSC; LCSC (none) -> C8490; MPN (none) -> LRC LBSS138LT1G
- R102, R105: Assembly (none) -> HAND; Distributor (none) -> LCSC; MPN (none) -> Yageo RC0603JR-0710KL
- R103: Assembly (none) -> HAND; Distributor (none) -> LCSC; MPN (none) -> Yageo RC0603JR-070RL
- R104, R93, R94, R95, R97: Assembly (none) -> HAND; Distributor (none) -> LCSC; MPN (none) -> Yageo RC0603JR-074K7L
- R106: Assembly (none) -> HAND; Distributor (none) -> LCSC; MPN (none) -> Yageo RC0603JR-07510RL
- R107: Assembly (none) -> HAND; Distributor (none) -> LCSC; MPN (none) -> Yageo RC0603JR-071ML
- R108: Assembly (none) -> HAND; Distributor (none) -> LCSC; MPN (none) -> Yageo RC0603FR-0759KL
- R109, R112: Assembly (none) -> HAND; Distributor (none) -> LCSC; MPN (none) -> Yageo RC0603FR-07100KL
- R110: Assembly (none) -> HAND; Distributor (none) -> LCSC; MPN (none) -> Yageo RC0603FR-0731K6L
- R111: Assembly (none) -> HAND; Distributor (none) -> LCSC; MPN (none) -> Yageo RC0603FR-0710KL
- R113: Assembly (none) -> HAND; Distributor (none) -> LCSC; MPN (none) -> Yageo RC0603FR-0720KL
- R96: Assembly (none) -> HAND; Distributor (none) -> LCSC; MPN (none) -> Yageo RC0603FR-072K49L
- U11: Assembly (none) -> HAND; Distributor (none) -> LCSC; MPN (none) -> Microchip 93LC46B-I/SN
- U12: Assembly (none) -> HAND; Distributor (none) -> LCSC; LCSC (none) -> C141836; MPN (none) -> TI TLV62569DBVR
- U15: Assembly (none) -> HAND; Distributor (none) -> LCSC; LCSC (none) -> C5219272; MPN (none) -> TI TPS62933FDRLR
- U9: Assembly (none) -> JLC; Distributor (none) -> LCSC; LCSC (none) -> C3013605; MPN (none) -> Realtek RTL8125BG-CG
- Y2: Assembly (none) -> HAND; Distributor (none) -> LCSC; MPN (none) -> Generic 25MHz (order-time equiv)
