File: sheets/ethernet.kicad_sch (KiCad schematic)
At the start: 58 parts, among them J8 2250504-1, Q36 BSS138, Q37 BSS138, Q38 BSS138, U11 93C46, U12 TLV62569DBVR, U15 TPS62933FDRLR, U9 RTL8125BG-CG, Y2 25MHz

Commit message: sch: Task 14 fixes — MPN/footprint agreement, numeric Q pins, durable approximation flags
Parts:
- C111, C113, C89, C92, C93: MPN Generic MLCC 100nF 0402 (Yageo/Murata/Samsung equiv, exact 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 -> Generic MLCC 100nF X7R 0603 (Yageo/Murata/Samsung equiv, ex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
Changed lines of the file:
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@@
 		(property "Datasheet" "" (at 250 20 0) (hide yes) (effects (font (size 1.27 1.27))))
 		(property "Assembly" "HAND" (at 250 20 0) (hide yes) (effects (font (size 1.27 1.27))))
-		(property "MPN" "Generic MLCC 100nF 0402 (Yageo/Murata/Samsung equiv, exact P/N TBD at order)" (at 250 20 0) (hide yes) (effects (font (size 1.27 1.27))))
+		(property "MPN" "Generic MLCC 100nF X7R 0603 (Yageo/Murata/Samsung equiv, exact P/N TBD at order)" (at 250 20 0) (hide yes) (effects (font (size 1.27 1.27))))
 		(property "Distributor" "LCSC" (at 250 20 0) (hide yes) (effects (font (size 1.27 1.27))))
 		(pin "1")
@@
 		(property "Datasheet" "" (at 250 65 0) (hide yes) (effects (font (size 1.27 1.27))))
 		(property "Assembly" "HAND" (at 250 65 0) (hide yes) (effects (font (size 1.27 1.27))))
-		(property "MPN" "Generic MLCC 100nF 0402 (Yageo/Murata/Samsung equiv, exact P/N TBD at order)" (at 250 65 0) (hide yes) (effects (font (size 1.27 1.27))))
+		(property "MPN" "Generic MLCC 100nF X7R 0603 (Yageo/Murata/Samsung equiv, exact P/N TBD at order)" (at 250 65 0) (hide yes) (effects (font (size 1.27 1.27))))
 		(property "Distributor" "LCSC" (at 250 65 0) (hide yes) (effects (font (size 1.27 1.27))))
 		(pin "1")
@@
 		(property "Datasheet" "" (at 250 80 0) (hide yes) (effects (font (size 1.27 1.27))))
 		(property "Assembly" "HAND" (at 250 80 0) (hide yes) (effects (font (size 1.27 1.27))))
-		(property "MPN" "Generic MLCC 100nF 0402 (Yageo/Murata/Samsung equiv, exact P/N TBD at order)" (at 250 80 0) (hide yes) (effects (font (size 1.27 1.27))))
+		(property "MPN" "Generic MLCC 100nF X7R 0603 (Yageo/Murata/Samsung equiv, exact P/N TBD at order)" (at 250 80 0) (hide yes) (effects (font (size 1.27 1.27))))
 		(property "Distributor" "LCSC" (at 250 80 0) (hide yes) (effects (font (size 1.27 1.27))))
 		(pin "1")
@@
 		(property "Datasheet" "" (at 30 200 0) (hide yes) (effects (font (size 1.27 1.27))))
 		(property "Assembly" "HAND" (at 30 200 0) (hide yes) (effects (font (size 1.27 1.27))))
-		(property "MPN" "Generic MLCC 100nF 0402 (Yageo/Murata/Samsung equiv, exact P/N TBD at order)" (at 30 200 0) (hide yes) (effects (font (size 1.27 1.27))))
+		(property "MPN" "Generic MLCC 100nF X7R 0603 (Yageo/Murata/Samsung equiv, exact P/N TBD at order)" (at 30 200 0) (hide yes) (effects (font (size 1.27 1.27))))
 		(property "Distributor" "LCSC" (at 30 200 0) (hide yes) (effects (font (size 1.27 1.27))))
 		(pin "1")
@@
 		(property "Datasheet" "" (at 110 190 0) (hide yes) (effects (font (size 1.27 1.27))))
 		(property "Assembly" "HAND" (at 110 190 0) (hide yes) (effects (font (size 1.27 1.27))))
-		(property "MPN" "Generic MLCC 100nF 0402 (Yageo/Murata/Samsung equiv, exact P/N TBD at order)" (at 110 190 0) (hide yes) (effects (font (size 1.27 1.27))))
+		(property "MPN" "Generic MLCC 100nF X7R 0603 (Yageo/Murata/Samsung equiv, exact P/N TBD at order)" (at 110 190 0) (hide yes) (effects (font (size 1.27 1.27))))
 		(property "Distributor" "LCSC" (at 110 190 0) (hide yes) (effects (font (size 1.27 1.27))))
 		(pin "1")
