File: sheets/sim.kicad_sch (KiCad schematic)
At the start: 0 parts

Commit message: sch: dual SIM + eSIM slot-2 override mux
Task 11: wire sheets/sim.kicad_sch (SIM1 direct nano-SIM + SIM2/eSIM
behind a TS3A27518E mux), author 4 new symbols (TS3A27518E, TPD4S009,
ST4SIM-200M, nano-SIM socket) in lib/sierra-to-usb.kicad_sym, extend
tools/netchecks.txt. Refdes remapped from the brief's stale placeholders
(collided with existing ethernet-sheet parts). NC/NO mux assignment and
the UIM2_DET_CTL override function both corrected vs. the brief's literal
wording per datasheet truth tables / DET-polarity physics (disclosed in
task-11-report.md). 0 ERC errors, all netchecks pass.
Parts:
- added C116, C117, C118, C119, C121, C122, C123, C124: 22pF, Capacitor_SMD:C_0402_1005Metric, symbol Device:C_Small
- added C120, C125, C126: 100nF, Capacitor_SMD:C_0402_1005Metric, symbol Device:C_Small
- added C127: 1uF, Capacitor_SMD:C_0603_1608Metric, symbol Device:C_Small
- added D27, D28: TPD4S009DBVR, Package_TO_SOT_SMD:SOT-23-6, symbol sierra-to-usb:TPD4S009
- added Q39: 2N7002, Package_TO_SOT_SMD:SOT-23, symbol Transistor_FET:2N7002
- added R114, R115, R116, R118, R119: 100k, Resistor_SMD:R_0603_1608Metric, symbol Device:R_Small
- added R117: 20k, Resistor_SMD:R_0603_1608Metric, symbol Device:R_Small
- added SIM1, SIM2: CSIM-H137-7P, sierra-to-usb:NanoSIM_JXTCONN_CSIM-H137-7P, symbol sierra-to-usb:JXTCONN_CSIM-H137-7P
- added U29: TS3A27518EPWR, Package_SO:TSSOP-24_4.4x7.8mm_P0.65mm, symbol sierra-to-usb:TS3A27518E
- added U30: ST4SIM-200M, sierra-to-usb:VFDFPN8_MFF2, symbol sierra-to-usb:ST4SIM-200M
Connections:
- new net +3V3: R114.2, R115.2, R118.2, U29.8 (VCC)
- new net GND: C116.2, C117.2, C118.2, C119.2, C120.2, C121.2, C122.2, C123.2, C124.2, C125.2, C126.2, C127.2, D27.2 (GND), D28.2 (GND), Q39.2 (S), R116.2, R119.2, SIM1.4 (GND), SIM1.6 (CD1), SIM2.4 (GND), SIM2.6 (CD1), U29.20 (EN), U29.5 (GND), U30.1 (GND)
- new net SIM_SEL: R116.1, U29.14 (IN2), U29.24 (IN1)
- new net UIM1_CLK: C117.1, D27.6 (D1-), SIM1.3 (CLK)
- new net UIM1_DET: C119.1, D27.4 (D2-), R114.1, SIM1.7 (CD2)
- new net UIM1_IO: C118.1, D27.3 (D2+), SIM1.5 (IO)
- new net UIM1_RST: C116.1, D27.1 (D1+), SIM1.2 (RST)
- new net UIM1_VDD: C120.1, D27.5 (VCC), SIM1.1 (VCC)
- new net UIM2E_CLK: U29.15 (NO3), U30.6 (CLK)
- new net UIM2E_DET: R118.1, U29.18 (NO5)
- new net UIM2E_IO: R117.1, U29.17 (NO4), U30.3 (I/O)
- new net UIM2E_RST: U29.13 (NO2), U30.7 (RESET)
- new net UIM2E_VDD: C126.1, C127.1, R117.2, U29.11 (NO1), U30.8 (VCC)
- new net UIM2S_CLK: C122.1, D28.6 (D1-), SIM2.3 (CLK), U29.23 (NC3)
- new net UIM2S_DET: C124.1, D28.4 (D2-), R115.1, SIM2.7 (CD2), U29.19 (NC5)
- new net UIM2S_IO: C123.1, D28.3 (D2+), SIM2.5 (IO), U29.21 (NC4)
- new net UIM2S_RST: C121.1, D28.1 (D1+), SIM2.2 (RST), U29.1 (NC2)
- new net UIM2S_VDD: C125.1, D28.5 (VCC), SIM2.1 (VCC), U29.2 (NC1)
- new net UIM2_CLK: U29.7 (COM3)
- new net UIM2_DET: Q39.3 (D), U29.10 (COM5)
- new net UIM2_DET_CTL: Q39.1 (G), R119.1
- new net UIM2_IO: U29.9 (COM4)
- new net UIM2_RST: U29.6 (COM2)
- new net UIM2_VDD: U29.4 (COM1)
- no-connect marks 0 -> 6
Other:
- note added: "Q39 (2N7002) + R115 (100k gate pull-down, reinforces RP2040's own internal pull-down default -- GP13/UIM2_DET_CTL blank-MCU default = OFF, no override) -- CORRECTED FUNCTION vs the brief's literal wording. Brief Step-3: 'Q8 2N7002 ... gate=UIM2_DET_CTL to assert present when eSIM active'. An N-channel FET can only pull its drain TOWARD GND -- i.e. it can only assert the verified 'grounded=absent'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"
- note added: "SIM1 direct to module UIM1_* (CN1 pins 36/30/32/34/66 per m2 sheet). D27=TPD4S009 ESD (4ch: RST/CLK/IO/DET) + 22pF/line + 100nF VDD bypass + 100k DET pull-up to +3V3, per both vendors' SIM reference circuits."
- note added: "SIM2 = physical slot 2, wired to U29's NC side (UIM2S_* -- sheet-local nets, not module-facing directly). D28=TPD4S009 ESD + 22pF/line + 100nF VDD bypass + 100k DET pull-up, same treatment as SIM1 (exposed card-edge contacts -- ESD/EMI risk on both physical sockets)."
- note added: "Task 11 -- dual SIM (SIM1/SIM2 physical nano-SIM sockets, ISO7816 5-wire) + eSIM (U30, ST4SIM-200M, on-board MFF2) slot-2 override mux (U29, TS3A27518E). SIM1 wired direct to module UIM1_*. UIM2_* (module) lands on U29's COM side; NC side (default, SIM_SEL pulled low) = physical SIM2 socket (UIM2S_*); NO side (SIM_SEL driven high) = eSIM branch (UIM2E_*). Refdes continue from the 325-component pr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"
- note added: "U29 TS3A27518E truth table (Table 8-1, EN=L): IN=L -> NCx<->COMx ON / NOx<->COMx OFF; IN=H -> NOx<->COMx ON / NCx<->COMx OFF. IN1/IN2 tied together onto SIM_SEL so both 3-channel banks move as one 6-channel 2:1 mux. VCC=+3V3 (module drives UIM2_VDD up to 3.0V typ; TS3A27518E requires VCC > max analog signal, abs-max VCC=4.6V, rec. op. 1.65-3.6V -- +3V3 clears both). VIH min=1.2V (Sec.6.3) << RP20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"
- note added: "U30 ST4SIM-200M (MFF2/VFDFPN8) pin table verified against ST data brief DB4082 Rev5 Fig.12/Table 4 (fetched via web.archive.org -- live st.com/mouser.com fetches were blocked/timed out during authoring, flagged in task-11-report.md). Powered from UIM2E_VDD (module-switched, via mux NO1), matching the ISOLATION/DOMAIN note -- NOT board +3V3. Decoupling = 100nF+1uF on VCC (Fig.6, datasheet-mandated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"

Commit message: sch: sim — remove 3V3 DET pull-ups (float=present per PTS), ch6 hygiene
Parts:
- removed R114, R115, R118: 100k, Resistor_SMD:R_0603_1608Metric, symbol Device:R_Small
Connections:
- net GND: now also U29.16 (NO6), U29.22 (NC6)
- no-connect marks 6 -> 4
Other:
- note added: "Q39 (2N7002) + R119 (100k gate pull-down, reinforces RP2040's own internal pull-down default -- GP13/UIM2_DET_CTL blank-MCU default = OFF, no override) -- CORRECTED FUNCTION vs the brief's literal wording. Brief Step-3: 'Q8 2N7002 ... gate=UIM2_DET_CTL to assert present when eSIM active'. An N-channel FET can only pull its drain TOWARD GND -- i.e. it can only assert the verified 'grounded=absent'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"
- note added: "SIM1 direct to module UIM1_* (CN1 pins 36/30/32/34/66 per m2 sheet). D27=TPD4S009 ESD (4ch: RST/CLK/IO/DET) + 22pF/line + 100nF VDD bypass. NO board-side DET pull-up (fix pass, 2026-07-15): CN1.66/UIM1_DET is a module-internal-pull-up two-state pin per the Sierra PTS (grounded=absent, floating=present) -- an added 100k-to-+3V3 pull-up put an undocumented third voltage on a likely-1.8V-domain pin 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"
- note added: "SIM2 = physical slot 2, wired to U29's NC side (UIM2S_* -- sheet-local nets, not module-facing directly). D28=TPD4S009 ESD + 22pF/line + 100nF VDD bypass, same treatment as SIM1 (exposed card-edge contacts -- ESD/EMI risk on both physical sockets). NO board-side DET pull-up (fix pass, 2026-07-15) -- same PTS two-state rationale as UIM1_DET; SIM2.CD2 floats through the mux's NC5 channel onto UIM2S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"
- note removed: "Q39 (2N7002) + R115 (100k gate pull-down, reinforces RP2040's own internal pull-down default -- GP13/UIM2_DET_CTL blank-MCU default = OFF, no override) -- CORRECTED FUNCTION vs the brief's literal wording. Brief Step-3: 'Q8 2N7002 ... gate=UIM2_DET_CTL to assert present when eSIM active'. An N-channel FET can only pull its drain TOWARD GND -- i.e. it can only assert the verified 'grounded=absent'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"
- note removed: "SIM1 direct to module UIM1_* (CN1 pins 36/30/32/34/66 per m2 sheet). D27=TPD4S009 ESD (4ch: RST/CLK/IO/DET) + 22pF/line + 100nF VDD bypass + 100k DET pull-up to +3V3, per both vendors' SIM reference circuits."
- note removed: "SIM2 = physical slot 2, wired to U29's NC side (UIM2S_* -- sheet-local nets, not module-facing directly). D28=TPD4S009 ESD + 22pF/line + 100nF VDD bypass + 100k DET pull-up, same treatment as SIM1 (exposed card-edge contacts -- ESD/EMI risk on both physical sockets)."
