File: sheets/sim.kicad_sch (KiCad schematic)
At the start: 22 parts, among them Q39 2N7002, U29 TS3A27518EPWR, U30 ST4SIM-200M

Commit message: sch: footprints + assembly-split BOM fields
Task 14: bind real footprints to all 363 BOM symbols, add Assembly/LCSC/MPN/
Distributor properties to every symbol, and close the accumulated
footprint_link_issues ERC deferral (148 -> 0).

- New fp-lib-table + lib/sierra-to-usb.pretty/ (15 custom footprints
  authored from real manufacturer drawings: magjack, MHF4, SMA edge,
  nano-SIM, MFF2 eSIM, M.2 socket, bridge rectifier, 2x PoE flyback
  inductors, TPS23730 VQFN-45, FDMC2523P, FOD817 gull-wing DIP-4, SK6805
  LED, PoE transformer, and a corrected full-24-pin USB-C receptacle for
  J1 -- the previously-bound stock footprint only exposed 6 of 24 pins).
- Fixed ~120 bare/stale/wrong-library-prefix Footprint strings project-wide.
- Assembly split: 12 JLC rows (all LCSC-backed), 351 HAND rows (MPN +
  Distributor on every one). Disclosed flip: U30 (eSIM) JLC->HAND per
  sourcing.md's own no-LCSC-listing flag, overriding the task's shorthand.
- Carry-forwards closed: D30 series R 1k->560R, INA226 MSOP-10->VSSOP-10
  (+EP-VIA), R39/R44 Kelvin-route note, JP1-3 solder-jumper footprints,
  SW2 silk note, 42x 0402->0603 hand-solder upgrades.
- New tools/check_footprints.py gate: Footprint/Assembly presence, JLC=>LCSC,
  and footprint-pad-count >= symbol-pin-count (parsed from real .kicad_mod
  files + netlist pin lists).
- Recovered sheets/mcu.kicad_sch from a pre-existing uncommitted data-loss
  state (44 symbols missing vs the Task 13 gate-approved commit) before
  applying any Task 14 edits.

Verification: check_footprints.py all-pass, check_nets.py all-pass
(connectivity untouched), kicad-cli sch erc 0 errors.

Two pre-existing issues disclosed but not fixed here (out of footprint-
assignment scope, documented in docs/verification.md and
docs/erc-waivers.md): J1's now-corrected footprint was masking a Task-7
error, and 7 refs (Q20,Q22-25,Q30,Q31) use letter-pinned generic FET/BJT
symbols that will show unmatched pins at PCB import regardless of
footprint choice -- flagge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
Parts:
- C116, C117, C118, C119, C121, C122, C123, C124: footprint Capacitor_SMD:C_0402_1005Metric -> Capacitor_SMD:C_0603_1608Metric; Assembly (none) -> HAND; Distributor (none) -> LCSC; MPN (none) -> Generic MLCC 22pF 0402 (Yageo/Murata/Samsung equiv, exact P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
- C120, C125, C126: footprint Capacitor_SMD:C_0402_1005Metric -> Capacitor_SMD:C_0603_1608Metric; Assembly (none) -> HAND; Distributor (none) -> LCSC; MPN (none) -> Generic MLCC 100nF 0402 (Yageo/Murata/Samsung equiv, exact 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
- C127: Assembly (none) -> HAND; Distributor (none) -> LCSC; MPN (none) -> Generic MLCC 1uF 0603 (Yageo/Murata/Samsung equiv, exact P/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
- D27, D28: Assembly (none) -> HAND; Distributor (none) -> LCSC; LCSC (none) -> C88032; MPN (none) -> TI TPD4S009DBVR
- Q39: Assembly (none) -> HAND; Distributor (none) -> LCSC; LCSC (none) -> C8545; MPN (none) -> 2N7002
- R116, R119: Assembly (none) -> HAND; Distributor (none) -> LCSC; MPN (none) -> Yageo RC0603JR-07100KL
- R117: Assembly (none) -> HAND; Distributor (none) -> LCSC; MPN (none) -> Yageo RC0603JR-0720KL
- SIM1, SIM2: Assembly (none) -> HAND; Distributor (none) -> LCSC; LCSC (none) -> C42420236; MPN (none) -> JXTCONN CSIM-H137-7P
- U29: Assembly (none) -> HAND; Distributor (none) -> LCSC; LCSC (none) -> C443721; MPN (none) -> TI TS3A27518EPWR
- U30: Assembly (none) -> HAND; Distributor (none) -> DigiKey; MPN (none) -> ST4SIM-200M
