File: sheets/sim.kicad_sch (KiCad schematic)
At the start: 22 parts, among them Q39 2N7002, U29 TS3A27518EPWR, U30 ST4SIM-200M

Commit message: sch: Task 14 fixes — MPN/footprint agreement, numeric Q pins, durable approximation flags
Parts:
- C116, C117, C118, C119, C121, C122, C123, C124: MPN Generic MLCC 22pF 0402 (Yageo/Murata/Samsung equiv, exact P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 -> Generic MLCC 22pF C0G 0603 (Yageo/Murata/Samsung equiv, exa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
- C120, C125, C126: MPN Generic MLCC 100nF 0402 (Yageo/Murata/Samsung equiv, exact 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 -> Generic MLCC 100nF X7R 0603 (Yageo/Murata/Samsung equiv, ex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
Changed lines of the file:
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@@
 		(property "Datasheet" "" (at 35 25 0) (hide yes) (effects (font (size 1.27 1.27))))
 		(property "Assembly" "HAND" (at 35 25 0) (hide yes) (effects (font (size 1.27 1.27))))
-		(property "MPN" "Generic MLCC 22pF 0402 (Yageo/Murata/Samsung equiv, exact P/N TBD at order)" (at 35 25 0) (hide yes) (effects (font (size 1.27 1.27))))
+		(property "MPN" "Generic MLCC 22pF C0G 0603 (Yageo/Murata/Samsung equiv, exact P/N TBD at order)" (at 35 25 0) (hide yes) (effects (font (size 1.27 1.27))))
 		(property "Distributor" "LCSC" (at 35 25 0) (hide yes) (effects (font (size 1.27 1.27))))
 		(pin "1")
@@
 		(property "Datasheet" "" (at 35 19 0) (hide yes) (effects (font (size 1.27 1.27))))
 		(property "Assembly" "HAND" (at 35 19 0) (hide yes) (effects (font (size 1.27 1.27))))
-		(property "MPN" "Generic MLCC 22pF 0402 (Yageo/Murata/Samsung equiv, exact P/N TBD at order)" (at 35 19 0) (hide yes) (effects (font (size 1.27 1.27))))
+		(property "MPN" "Generic MLCC 22pF C0G 0603 (Yageo/Murata/Samsung equiv, exact P/N TBD at order)" (at 35 19 0) (hide yes) (effects (font (size 1.27 1.27))))
 		(property "Distributor" "LCSC" (at 35 19 0) (hide yes) (effects (font (size 1.27 1.27))))
 		(pin "1")
@@
 		(property "Datasheet" "" (at 35 13 0) (hide yes) (effects (font (size 1.27 1.27))))
 		(property "Assembly" "HAND" (at 35 13 0) (hide yes) (effects (font (size 1.27 1.27))))
-		(property "MPN" "Generic MLCC 22pF 0402 (Yageo/Murata/Samsung equiv, exact P/N TBD at order)" (at 35 13 0) (hide yes) (effects (font (size 1.27 1.27))))
+		(property "MPN" "Generic MLCC 22pF C0G 0603 (Yageo/Murata/Samsung equiv, exact P/N TBD at order)" (at 35 13 0) (hide yes) (effects (font (size 1.27 1.27))))
 		(property "Distributor" "LCSC" (at 35 13 0) (hide yes) (effects (font (size 1.27 1.27))))
 		(pin "1")
@@
 		(property "Datasheet" "" (at 35 7 0) (hide yes) (effects (font (size 1.27 1.27))))
 		(property "Assembly" "HAND" (at 35 7 0) (hide yes) (effects (font (size 1.27 1.27))))
-		(property "MPN" "Generic MLCC 22pF 0402 (Yageo/Murata/Samsung equiv, exact P/N TBD at order)" (at 35 7 0) (hide yes) (effects (font (size 1.27 1.27))))
+		(property "MPN" "Generic MLCC 22pF C0G 0603 (Yageo/Murata/Samsung equiv, exact P/N TBD at order)" (at 35 7 0) (hide yes) (effects (font (size 1.27 1.27))))
 		(property "Distributor" "LCSC" (at 35 7 0) (hide yes) (effects (font (size 1.27 1.27))))
 		(pin "1")
@@
 		(property "Datasheet" "" (at 35 1 0) (hide yes) (effects (font (size 1.27 1.27))))
 		(property "Assembly" "HAND" (at 35 1 0) (hide yes) (effects (font (size 1.27 1.27))))
-		(property "MPN" "Generic MLCC 100nF 0402 (Yageo/Murata/Samsung equiv, exact P/N TBD at order)" (at 35 1 0) (hide yes) (effects (font (size 1.27 1.27))))
+		(property "MPN" "Generic MLCC 100nF X7R 0603 (Yageo/Murata/Samsung equiv, exact P/N TBD at order)" (at 35 1 0) (hide yes) (effects (font (size 1.27 1.27))))
 		(property "Distributor" "LCSC" (at 35 1 0) (hide yes) (effects (font (size 1.27 1.27))))
 		(pin "1")
@@
 		(property "Datasheet" "" (at 35 125 0) (hide yes) (effects (font (size 1.27 1.27))))
 		(property "Assembly" "HAND" (at 35 125 0) (hide yes) (effects (font (size 1.27 1.27))))
-		(property "MPN" "Generic MLCC 22pF 0402 (Yageo/Murata/Samsung equiv, exact P/N TBD at order)" (at 35 125 0) (hide yes) (effects (font (size 1.27 1.27))))
+		(property "MPN" "Generic MLCC 22pF C0G 0603 (Yageo/Murata/Samsung equiv, exact P/N TBD at order)" (at 35 125 0) (hide yes) (effects (font (size 1.27 1.27))))
 		(property "Distributor" "LCSC" (at 35 125 0) (hide yes) (effects (font (size 1.27 1.27))))
 		(pin "1")
@@
 		(property "Datasheet" "" (at 35 119 0) (hide yes) (effects (font (size 1.27 1.27))))
 		(property "Assembly" "HAND" (at 35 119 0) (hide yes) (effects (font (size 1.27 1.27))))
-		(property "MPN" "Generic MLCC 22pF 0402 (Yageo/Murata/Samsung equiv, exact P/N TBD at order)" (at 35 119 0) (hide yes) (effects (font (size 1.27 1.27))))
+		(property "MPN" "Generic MLCC 22pF C0G 0603 (Yageo/Murata/Samsung equiv, exact P/N TBD at order)" (at 35 119 0) (hide yes) (effects (font (size 1.27 1.27))))
 		(property "Distributor" "LCSC" (at 35 119 0) (hide yes) (effects (font (size 1.27 1.27))))
 		(pin "1")
@@
 		(property "Datasheet" "" (at 35 113 0) (hide yes) (effects (font (size 1.27 1.27))))
 		(property "Assembly" "HAND" (at 35 113 0) (hide yes) (effects (font (size 1.27 1.27))))
-		(property "MPN" "Generic MLCC 22pF 0402 (Yageo/Murata/Samsung equiv, exact P/N TBD at order)" (at 35 113 0) (hide yes) (effects (font (size 1.27 1.27))))
+		(property "MPN" "Generic MLCC 22pF C0G 0603 (Yageo/Murata/Samsung equiv, exact P/N TBD at order)" (at 35 113 0) (hide yes) (effects (font (size 1.27 1.27))))
 		(property "Distributor" "LCSC" (at 35 113 0) (hide yes) (effects (font (size 1.27 1.27))))
 		(pin "1")
@@
 		(property "Datasheet" "" (at 35 107 0) (hide yes) (effects (font (size 1.27 1.27))))
 		(property "Assembly" "HAND" (at 35 107 0) (hide yes) (effects (font (size 1.27 1.27))))
-		(property "MPN" "Generic MLCC 22pF 0402 (Yageo/Murata/Samsung equiv, exact P/N TBD at order)" (at 35 107 0) (hide yes) (effects (font (size 1.27 1.27))))
+		(property "MPN" "Generic MLCC 22pF C0G 0603 (Yageo/Murata/Samsung equiv, exact P/N TBD at order)" (at 35 107 0) (hide yes) (effects (font (size 1.27 1.27))))
 		(property "Distributor" "LCSC" (at 35 107 0) (hide yes) (effects (font (size 1.27 1.27))))
 		(pin "1")
@@
 		(property "Datasheet" "" (at 35 101 0) (hide yes) (effects (font (size 1.27 1.27))))
 		(property "Assembly" "HAND" (at 35 101 0) (hide yes) (effects (font (size 1.27 1.27))))
-		(property "MPN" "Generic MLCC 100nF 0402 (Yageo/Murata/Samsung equiv, exact P/N TBD at order)" (at 35 101 0) (hide yes) (effects (font (size 1.27 1.27))))
+		(property "MPN" "Generic MLCC 100nF X7R 0603 (Yageo/Murata/Samsung equiv, exact P/N TBD at order)" (at 35 101 0) (hide yes) (effects (font (size 1.27 1.27))))
 		(property "Distributor" "LCSC" (at 35 101 0) (hide yes) (effects (font (size 1.27 1.27))))
 		(pin "1")
@@
 		(property "Datasheet" "" (at 245 45 0) (hide yes) (effects (font (size 1.27 1.27))))
 		(property "Assembly" "HAND" (at 245 45 0) (hide yes) (effects (font (size 1.27 1.27))))
-		(property "MPN" "Generic MLCC 100nF 0402 (Yageo/Murata/Samsung equiv, exact P/N TBD at order)" (at 245 45 0) (hide yes) (effects (font (size 1.27 1.27))))
+		(property "MPN" "Generic MLCC 100nF X7R 0603 (Yageo/Murata/Samsung equiv, exact P/N TBD at order)" (at 245 45 0) (hide yes) (effects (font (size 1.27 1.27))))
 		(property "Distributor" "LCSC" (at 245 45 0) (hide yes) (effects (font (size 1.27 1.27))))
 		(pin "1")
