File: sheets/rf.kicad_sch (KiCad schematic)
At the start: 0 parts

Commit message: sch: 5x MHF4-to-SMA RF breakouts
Parts:
- added J10, J12, J14, J16, J18: BWSMA-KE-Z001, sierra-to-usb:SMA_EdgeMount_BWSMA-KE-Z001, symbol Connector:Conn_Coaxial
- added J11, J13, J15, J17, J9: CONMHF4-SMD-G-T, sierra-to-usb:MHF4_TE_CONMHF4-SMD-G-T, symbol Connector:Conn_Coaxial
Connections:
- new net ANT0: J10.1 (In), J9.1 (In)
- new net ANT1: J11.1 (In), J12.1 (In)
- new net ANT2: J13.1 (In), J14.1 (In)
- new net ANT3: J15.1 (In), J16.1 (In)
- new net GND: J10.2 (Ext), J11.2 (Ext), J12.2 (Ext), J13.2 (Ext), J14.2 (Ext), J15.2 (Ext), J16.2 (Ext), J17.2 (Ext), J18.2 (Ext), J9.2 (Ext)
- new net GNSS: J17.1 (In), J18.1 (In)
Other:
- note added: "50 ohm CPWG, via-fenced, keep runs short -- see plan Task 18; label silks ANT0-3/GNSS at both connectors. (ASCII-substituted for the project's plain-ASCII sheet convention: "ohm" for the Omega symbol, "--" for the em dash -- semantics unchanged.)"
- note added: "Task 12 -- 5x MHF4 (SMT receptacle) -> SMA (edge jack) RF antenna breakouts. Pure passive: signal center pin (pin 1) net-to-net per pair, shield/ground pin (pin 2) tied to GND at both ends. Nets ANT0/ANT1/ANT2/ANT3/GNSS, netclass RF_50 (patterns "ANT*"/"GNSS", declared project-file Task 3, unmodified here -- verified names match). Refdes remap (brief's placeholder J5-J9 MHF4 / J10-J14 SMA, offset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"
