File: sheets/rf.kicad_sch (KiCad schematic)
At the start: 10 parts, among them J10 BWSMA-KE-Z001, J11 CONMHF4-SMD-G-T, J12 BWSMA-KE-Z001, J13 CONMHF4-SMD-G-T, J14 BWSMA-KE-Z001, J15 CONMHF4-SMD-G-T, J16 BWSMA-KE-Z001, J17 CONMHF4-SMD-G-T, J18 BWSMA-KE-Z001, J9 CONMHF4-SMD-G-T

Commit message: sch: footprints + assembly-split BOM fields
Task 14: bind real footprints to all 363 BOM symbols, add Assembly/LCSC/MPN/
Distributor properties to every symbol, and close the accumulated
footprint_link_issues ERC deferral (148 -> 0).

- New fp-lib-table + lib/sierra-to-usb.pretty/ (15 custom footprints
  authored from real manufacturer drawings: magjack, MHF4, SMA edge,
  nano-SIM, MFF2 eSIM, M.2 socket, bridge rectifier, 2x PoE flyback
  inductors, TPS23730 VQFN-45, FDMC2523P, FOD817 gull-wing DIP-4, SK6805
  LED, PoE transformer, and a corrected full-24-pin USB-C receptacle for
  J1 -- the previously-bound stock footprint only exposed 6 of 24 pins).
- Fixed ~120 bare/stale/wrong-library-prefix Footprint strings project-wide.
- Assembly split: 12 JLC rows (all LCSC-backed), 351 HAND rows (MPN +
  Distributor on every one). Disclosed flip: U30 (eSIM) JLC->HAND per
  sourcing.md's own no-LCSC-listing flag, overriding the task's shorthand.
- Carry-forwards closed: D30 series R 1k->560R, INA226 MSOP-10->VSSOP-10
  (+EP-VIA), R39/R44 Kelvin-route note, JP1-3 solder-jumper footprints,
  SW2 silk note, 42x 0402->0603 hand-solder upgrades.
- New tools/check_footprints.py gate: Footprint/Assembly presence, JLC=>LCSC,
  and footprint-pad-count >= symbol-pin-count (parsed from real .kicad_mod
  files + netlist pin lists).
- Recovered sheets/mcu.kicad_sch from a pre-existing uncommitted data-loss
  state (44 symbols missing vs the Task 13 gate-approved commit) before
  applying any Task 14 edits.

Verification: check_footprints.py all-pass, check_nets.py all-pass
(connectivity untouched), kicad-cli sch erc 0 errors.

Two pre-existing issues disclosed but not fixed here (out of footprint-
assignment scope, documented in docs/verification.md and
docs/erc-waivers.md): J1's now-corrected footprint was masking a Task-7
error, and 7 refs (Q20,Q22-25,Q30,Q31) use letter-pinned generic FET/BJT
symbols that will show unmatched pins at PCB import regardless of
footprint choice -- flagge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
Parts:
- J10, J12, J14, J16, J18: Assembly (none) -> HAND; Distributor (none) -> LCSC; LCSC (none) -> C496549; MPN (none) -> BAT Wireless BWSMA-KE-Z001
- J11, J13, J15, J17, J9: Assembly (none) -> JLC; Distributor (none) -> LCSC; LCSC (none) -> C18221168; MPN (none) -> TE CONMHF4-SMD-G-T
Changed lines of the file:
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@@
 		(property "Footprint" "sierra-to-usb:MHF4_TE_CONMHF4-SMD-G-T" (at 20 30 0) (hide yes) (effects (font (size 1.27 1.27))))
 		(property "Datasheet" "https://www.lcsc.com/product-detail/C18221168.html" (at 20 30 0) (hide yes) (effects (font (size 1.27 1.27))))
+		(property "Assembly" "JLC" (at 20 30 0) (hide yes) (effects (font (size 1.27 1.27))))
+		(property "LCSC" "C18221168" (at 20 30 0) (hide yes) (effects (font (size 1.27 1.27))))
+		(property "MPN" "TE CONMHF4-SMD-G-T" (at 20 30 0) (hide yes) (effects (font (size 1.27 1.27))))
+		(property "Distributor" "LCSC" (at 20 30 0) (hide yes) (effects (font (size 1.27 1.27))))
 		(pin "1")
 		(pin "2")
@@
 		(property "Footprint" "sierra-to-usb:SMA_EdgeMount_BWSMA-KE-Z001" (at 70 30 0) (hide yes) (effects (font (size 1.27 1.27))))
 		(property "Datasheet" "https://www.lcsc.com/product-detail/C496549.html" (at 70 30 0) (hide yes) (effects (font (size 1.27 1.27))))
+		(property "Assembly" "HAND" (at 70 30 0) (hide yes) (effects (font (size 1.27 1.27))))
+		(property "LCSC" "C496549" (at 70 30 0) (hide yes) (effects (font (size 1.27 1.27))))
+		(property "MPN" "BAT Wireless BWSMA-KE-Z001" (at 70 30 0) (hide yes) (effects (font (size 1.27 1.27))))
+		(property "Distributor" "LCSC" (at 70 30 0) (hide yes) (effects (font (size 1.27 1.27))))
 		(pin "1")
 		(pin "2")
@@
 		(property "Footprint" "sierra-to-usb:MHF4_TE_CONMHF4-SMD-G-T" (at 20 50 0) (hide yes) (effects (font (size 1.27 1.27))))
 		(property "Datasheet" "https://www.lcsc.com/product-detail/C18221168.html" (at 20 50 0) (hide yes) (effects (font (size 1.27 1.27))))
+		(property "Assembly" "JLC" (at 20 50 0) (hide yes) (effects (font (size 1.27 1.27))))
+		(property "LCSC" "C18221168" (at 20 50 0) (hide yes) (effects (font (size 1.27 1.27))))
+		(property "MPN" "TE CONMHF4-SMD-G-T" (at 20 50 0) (hide yes) (effects (font (size 1.27 1.27))))
+		(property "Distributor" "LCSC" (at 20 50 0) (hide yes) (effects (font (size 1.27 1.27))))
 		(pin "1")
 		(pin "2")
@@
 		(property "Footprint" "sierra-to-usb:SMA_EdgeMount_BWSMA-KE-Z001" (at 70 50 0) (hide yes) (effects (font (size 1.27 1.27))))
 		(property "Datasheet" "https://www.lcsc.com/product-detail/C496549.html" (at 70 50 0) (hide yes) (effects (font (size 1.27 1.27))))
+		(property "Assembly" "HAND" (at 70 50 0) (hide yes) (effects (font (size 1.27 1.27))))
+		(property "LCSC" "C496549" (at 70 50 0) (hide yes) (effects (font (size 1.27 1.27))))
+		(property "MPN" "BAT Wireless BWSMA-KE-Z001" (at 70 50 0) (hide yes) (effects (font (size 1.27 1.27))))
+		(property "Distributor" "LCSC" (at 70 50 0) (hide yes) (effects (font (size 1.27 1.27))))
 		(pin "1")
 		(pin "2")
@@
 		(property "Footprint" "sierra-to-usb:MHF4_TE_CONMHF4-SMD-G-T" (at 20 70 0) (hide yes) (effects (font (size 1.27 1.27))))
 		(property "Datasheet" "https://www.lcsc.com/product-detail/C18221168.html" (at 20 70 0) (hide yes) (effects (font (size 1.27 1.27))))
+		(property "Assembly" "JLC" (at 20 70 0) (hide yes) (effects (font (size 1.27 1.27))))
+		(property "LCSC" "C18221168" (at 20 70 0) (hide yes) (effects (font (size 1.27 1.27))))
+		(property "MPN" "TE CONMHF4-SMD-G-T" (at 20 70 0) (hide yes) (effects (font (size 1.27 1.27))))
+		(property "Distributor" "LCSC" (at 20 70 0) (hide yes) (effects (font (size 1.27 1.27))))
 		(pin "1")
 		(pin "2")
@@
 		(property "Footprint" "sierra-to-usb:SMA_EdgeMount_BWSMA-KE-Z001" (at 70 70 0) (hide yes) (effects (font (size 1.27 1.27))))
 		(property "Datasheet" "https://www.lcsc.com/product-detail/C496549.html" (at 70 70 0) (hide yes) (effects (font (size 1.27 1.27))))
+		(property "Assembly" "HAND" (at 70 70 0) (hide yes) (effects (font (size 1.27 1.27))))
+		(property "LCSC" "C496549" (at 70 70 0) (hide yes) (effects (font (size 1.27 1.27))))
+		(property "MPN" "BAT Wireless BWSMA-KE-Z001" (at 70 70 0) (hide yes) (effects (font (size 1.27 1.27))))
+		(property "Distributor" "LCSC" (at 70 70 0) (hide yes) (effects (font (size 1.27 1.27))))
 		(pin "1")
 		(pin "2")
@@
 		(property "Footprint" "sierra-to-usb:MHF4_TE_CONMHF4-SMD-G-T" (at 20 90 0) (hide yes) (effects (font (size 1.27 1.27))))
 		(property "Datasheet" "https://www.lcsc.com/product-detail/C18221168.html" (at 20 90 0) (hide yes) (effects (font (size 1.27 1.27))))
+		(property "Assembly" "JLC" (at 20 90 0) (hide yes) (effects (font (size 1.27 1.27))))
+		(property "LCSC" "C18221168" (at 20 90 0) (hide yes) (effects (font (size 1.27 1.27))))
+		(property "MPN" "TE CONMHF4-SMD-G-T" (at 20 90 0) (hide yes) (effects (font (size 1.27 1.27))))
+		(property "Distributor" "LCSC" (at 20 90 0) (hide yes) (effects (font (size 1.27 1.27))))
 		(pin "1")
 		(pin "2")
@@
 		(property "Footprint" "sierra-to-usb:SMA_EdgeMount_BWSMA-KE-Z001" (at 70 90 0) (hide yes) (effects (font (size 1.27 1.27))))
 		(property "Datasheet" "https://www.lcsc.com/product-detail/C496549.html" (at 70 90 0) (hide yes) (effects (font (size 1.27 1.27))))
+		(property "Assembly" "HAND" (at 70 90 0) (hide yes) (effects (font (size 1.27 1.27))))
+		(property "LCSC" "C496549" (at 70 90 0) (hide yes) (effects (font (size 1.27 1.27))))
+		(property "MPN" "BAT Wireless BWSMA-KE-Z001" (at 70 90 0) (hide yes) (effects (font (size 1.27 1.27))))
+		(property "Distributor" "LCSC" (at 70 90 0) (hide yes) (effects (font (size 1.27 1.27))))
 		(pin "1")
 		(pin "2")
@@
 		(property "Footprint" "sierra-to-usb:MHF4_TE_CONMHF4-SMD-G-T" (at 20 110 0) (hide yes) (effects (font (size 1.27 1.27))))
 		(property "Datasheet" "https://www.lcsc.com/product-detail/C18221168.html" (at 20 110 0) (hide yes) (effects (font (size 1.27 1.27))))
+		(property "Assembly" "JLC" (at 20 110 0) (hide yes) (effects (font (size 1.27 1.27))))
+		(property "LCSC" "C18221168" (at 20 110 0) (hide yes) (effects (font (size 1.27 1.27))))
+		(property "MPN" "TE CONMHF4-SMD-G-T" (at 20 110 0) (hide yes) (effects (font (size 1.27 1.27))))
+		(property "Distributor" "LCSC" (at 20 110 0) (hide yes) (effects (font (size 1.27 1.27))))
 		(pin "1")
 		(pin "2")
@@
 		(property "Footprint" "sierra-to-usb:SMA_EdgeMount_BWSMA-KE-Z001" (at 70 110 0) (hide yes) (effects (font (size 1.27 1.27))))
 		(property "Datasheet" "https://www.lcsc.com/product-detail/C496549.html" (at 70 110 0) (hide yes) (effects (font (size 1.27 1.27))))
-		(pin "1")
-		(pin "2")
+		(property "Assembly" "HAND" (at 70 110 0) (hide yes) (effects (font (size 1.27 1.27))))
+		(property "LCSC" "C496549" (at 70 110 0) (hide yes) (effects (font (size 1.27 1.27))))
+		(property "MPN" "BAT Wireless BWSMA-KE-Z001" (at 70 110 0) (hide yes) (effects (font (size 1.27 1.27))))
+		(property "Distributor" "LCSC" (at 70 110 0) (hide yes) (effects (font (size 1.27 1.27))))
+		(pin "1")
+		(pin "2")
