File: sheets/usb3_data.kicad_sch (KiCad schematic)
At the start: 16 parts, among them J1 TYPE-C-31-M-17, U1 HD3SS3220RNHR, U4 AP2112K-3.3TRG1

Commit message: sch: footprints + assembly-split BOM fields
Task 14: bind real footprints to all 363 BOM symbols, add Assembly/LCSC/MPN/
Distributor properties to every symbol, and close the accumulated
footprint_link_issues ERC deferral (148 -> 0).

- New fp-lib-table + lib/sierra-to-usb.pretty/ (15 custom footprints
  authored from real manufacturer drawings: magjack, MHF4, SMA edge,
  nano-SIM, MFF2 eSIM, M.2 socket, bridge rectifier, 2x PoE flyback
  inductors, TPS23730 VQFN-45, FDMC2523P, FOD817 gull-wing DIP-4, SK6805
  LED, PoE transformer, and a corrected full-24-pin USB-C receptacle for
  J1 -- the previously-bound stock footprint only exposed 6 of 24 pins).
- Fixed ~120 bare/stale/wrong-library-prefix Footprint strings project-wide.
- Assembly split: 12 JLC rows (all LCSC-backed), 351 HAND rows (MPN +
  Distributor on every one). Disclosed flip: U30 (eSIM) JLC->HAND per
  sourcing.md's own no-LCSC-listing flag, overriding the task's shorthand.
- Carry-forwards closed: D30 series R 1k->560R, INA226 MSOP-10->VSSOP-10
  (+EP-VIA), R39/R44 Kelvin-route note, JP1-3 solder-jumper footprints,
  SW2 silk note, 42x 0402->0603 hand-solder upgrades.
- New tools/check_footprints.py gate: Footprint/Assembly presence, JLC=>LCSC,
  and footprint-pad-count >= symbol-pin-count (parsed from real .kicad_mod
  files + netlist pin lists).
- Recovered sheets/mcu.kicad_sch from a pre-existing uncommitted data-loss
  state (44 symbols missing vs the Task 13 gate-approved commit) before
  applying any Task 14 edits.

Verification: check_footprints.py all-pass, check_nets.py all-pass
(connectivity untouched), kicad-cli sch erc 0 errors.

Two pre-existing issues disclosed but not fixed here (out of footprint-
assignment scope, documented in docs/verification.md and
docs/erc-waivers.md): J1's now-corrected footprint was masking a Task-7
error, and 7 refs (Q20,Q22-25,Q30,Q31) use letter-pinned generic FET/BJT
symbols that will show unmatched pins at PCB import regardless of
footprint choice -- flagge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
Parts:
- C58, C59: Assembly (none) -> HAND; Distributor (none) -> LCSC; MPN (none) -> Generic MLCC 220nF 0603 (Yageo/Murata/Samsung equiv, exact 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
- C60, C61: Assembly (none) -> HAND; Distributor (none) -> LCSC; MPN (none) -> Generic MLCC 1uF/16V 0603 (Yageo/Murata/Samsung equiv, exac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
- C62: Assembly (none) -> HAND; Distributor (none) -> LCSC; MPN (none) -> Generic MLCC 1nF 0603 (Yageo/Murata/Samsung equiv, exact P/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
- D20, D21, D22: Assembly (none) -> HAND; Distributor (none) -> LCSC; LCSC (none) -> C558427; MPN (none) -> TI TPD4EUSB30DQAR
- D23: Assembly (none) -> HAND; Distributor (none) -> LCSC; LCSC (none) -> C138714; MPN (none) -> TI TPD4E05U06DQAR
- D24: footprint Diode_SMB:D_SMB -> Diode_SMD:D_SMB; Assembly (none) -> HAND; Distributor (none) -> LCSC; LCSC (none) -> C98802; MPN (none) -> ST SMAJ5.0A-TR
- J1: footprint Connector_USB:USB_C_Receptacle_HRO_TYPE-C-31-M-17 -> sierra-to-usb:USB_C_Receptacle_HRO_TYPE-C-31-M-17_Full24P; Assembly (none) -> HAND; Distributor (none) -> LCSC; LCSC (none) -> C283540; MPN (none) -> HRO TYPE-C-31-M-17
- R69: Assembly (none) -> HAND; Distributor (none) -> LCSC; MPN (none) -> Yageo RC0603FR-07900KL
- R70: Assembly (none) -> HAND; Distributor (none) -> LCSC; MPN (none) -> Yageo RC0603JR-071ML
- R71: Assembly (none) -> HAND; Distributor (none) -> LCSC; MPN (none) -> Yageo RC0603JR-07200KL
- U1: footprint Package_DFN_QFN:HD3SS3220_RNH0030A -> Package_DFN_QFN:Texas_RNH0030A_WQFN-30-1EP_2.5x4.5mm_P0.4mm_EP1.2x3.2mm; Assembly (none) -> JLC; Distributor (none) -> LCSC; LCSC (none) -> C165155; MPN (none) -> TI HD3SS3220RNHR
- U4: Assembly (none) -> HAND; Distributor (none) -> LCSC; LCSC (none) -> C51118; MPN (none) -> Diodes AP2112K-3.3TRG1

Commit message: sch: fix J1's MPN — pinned part was a 6-pin detector switch, not 24-pin USB3
Follow-up to the previous commit: the J1 footprint fix surfaced a deeper
problem than a wrong footprint. HRO TYPE-C-31-M-17 (LCSC C283540, pinned at
Task 7) is titled "DETECTOR SWITCHS" in its own manufacturer datasheet and
is a genuine 6-pin CC/VBUS/GND-only receptacle -- it cannot carry USB3 data
regardless of which footprint is bound to it. Task 7's footprint-filename
match was coincidental, not a real part match.

Re-pinned J1 to HRO TYPE-C-31-M-04 (LCSC C129018), the real 24-pin
full-featured part in the same family, whose datasheet pin table matches
the project's USB_C_Receptacle_USB3.2_24P symbol pin-for-pin. Updated
docs/sourcing.md, J1's Value/MPN/LCSC/Datasheet schematic properties
(text-only, no connectivity change), and renamed/relabeled the custom
footprint to sierra-to-usb:USB_C_Receptacle_HRO_TYPE-C-31-M-04 (25 pads,
matches the symbol's 25 pins).

Re-verified clean: check_footprints.py all-pass, check_nets.py all-pass,
kicad-cli sch erc 0 errors.

Co-Authored-By: Claude Fable 5 <noreply@anthropic.com>
Parts:
- J1: value TYPE-C-31-M-17 -> TYPE-C-31-M-04; footprint sierra-to-usb:USB_C_Receptacle_HRO_TYPE-C-31-M-17_Full24P -> sierra-to-usb:USB_C_Receptacle_HRO_TYPE-C-31-M-04; LCSC C283540 -> C129018; MPN HRO TYPE-C-31-M-17 -> HRO TYPE-C-31-M-04
Changed lines of the file:
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@@
 		(fields_autoplaced yes)
 		(property "Reference" "J1" (at 17 57 0) (effects (font (size 1.27 1.27))))
-		(property "Value" "TYPE-C-31-M-17" (at 17 63 0) (effects (font (size 1.27 1.27))))
-		(property "Footprint" "sierra-to-usb:USB_C_Receptacle_HRO_TYPE-C-31-M-17_Full24P" (at 20 60 0) (hide yes) (effects (font (size 1.27 1.27))))
-		(property "Datasheet" "" (at 20 60 0) (hide yes) (effects (font (size 1.27 1.27))))
+		(property "Value" "TYPE-C-31-M-04" (at 17 63 0) (effects (font (size 1.27 1.27))))
+		(property "Footprint" "sierra-to-usb:USB_C_Receptacle_HRO_TYPE-C-31-M-04" (at 20 60 0) (hide yes) (effects (font (size 1.27 1.27))))
+		(property "Datasheet" "https://datasheet.lcsc.com/datasheet/pdf/c25d4978cafd1404c08bb98baca46f59.pdf" (at 20 60 0) (hide yes) (effects (font (size 1.27 1.27))))
 		(property "Assembly" "HAND" (at 20 60 0) (hide yes) (effects (font (size 1.27 1.27))))
-		(property "LCSC" "C283540" (at 20 60 0) (hide yes) (effects (font (size 1.27 1.27))))
-		(property "MPN" "HRO TYPE-C-31-M-17" (at 20 60 0) (hide yes) (effects (font (size 1.27 1.27))))
+		(property "LCSC" "C129018" (at 20 60 0) (hide yes) (effects (font (size 1.27 1.27))))
+		(property "MPN" "HRO TYPE-C-31-M-04" (at 20 60 0) (hide yes) (effects (font (size 1.27 1.27))))
 		(property "Distributor" "LCSC" (at 20 60 0) (hide yes) (effects (font (size 1.27 1.27))))
 		(pin "A1")
