File: sheets/power_input.kicad_sch (KiCad schematic)
At the start: 110 parts, among them J2 TYPE-C-31-M-12, Q20 FDMS86250, Q21 FDMC2523P, Q22 BSC057N08NS3 G, Q23 BSC057N08NS3 G, Q24 FCX493TA, Q25 FCX493TA, Q30 IRLR7843TRPBF, Q31 IRLR7843TRPBF, T1 750313355, U10 TPS23730RMTR, U19 LM5050MKX-1/NOPB, U2 CH224K, U20 TCMT1107, U21 LM5050MKX-1/NOPB, U22 TL431IDBVR, U23 FOD817DS

Commit message: sch: Task 14 fixes — MPN/footprint agreement, numeric Q pins, durable approximation flags
Parts:
- Q20, Q22, Q23: symbol Device:Q_NMOS -> sierra-to-usb:Q_NMOS_TDSON_PQFN
- Q24, Q25: symbol Device:Q_NPN -> sierra-to-usb:Q_NPN_SOT89
- Q30, Q31: symbol Device:Q_NMOS -> sierra-to-usb:Q_NMOS_DPAK
Connections:
- net +12V: now also Q30.2 (D), Q31.2 (D); no longer Q30.D, Q31.D
- net +12V_POE: now also Q31.3 (S); no longer Q31.S
- net GND: now also Q22.1 (S), Q23.1 (S); no longer Q22.S, Q23.S
- net N_CS_SNS: now also Q20.1 (S); no longer Q20.S
- net N_GATE_Q: now also Q20.4 (G); no longer Q20.G
- net N_Q22_G: now also Q22.4 (G), Q24.3 (E); no longer Q22.G, Q24.E
- net N_Q23_G: now also Q23.4 (G), Q25.3 (E); no longer Q23.G, Q25.E
- net N_Q24_B: now also Q24.1 (B); no longer Q24.B
- net N_Q25_B: now also Q25.1 (B); no longer Q25.B
- net N_SEC_RTN: now also Q22.5 (D), Q25.2 (C); no longer Q22.D, Q25.C
- net N_SEC_SW: now also Q23.5 (D), Q24.2 (C); no longer Q23.D, Q24.C
- net N_SW: now also Q20.5 (D); no longer Q20.D
- net N_U19_GATE: now also Q30.1 (G); no longer Q30.G
- net N_U21_GATE: now also Q31.1 (G); no longer Q31.G
- net VBUS_PD: now also Q30.3 (S); no longer Q30.S
Changed lines of the file:
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@@
 	)
 	(symbol
-		(lib_id "Device:Q_NMOS")
+		(lib_id "sierra-to-usb:Q_NMOS_TDSON_PQFN")
 		(at 350 60 0)
 		(unit 1)
@@
 		(property "Distributor" "DigiKey" (at 350 60 0) (hide yes) (effects (font (size 1.27 1.27))))
 		(property "EP-VIA" "yes" (at 350 60 0) (hide yes) (effects (font (size 1.27 1.27))))
-		(pin "D"
-		)
-		(pin "G"
-		)
-		(pin "S"
+		(pin "5"
+		)
+		(pin "4"
+		)
+		(pin "1"
 		)
 		(instances
@@
 	)
 	(symbol
-		(lib_id "Device:Q_NMOS")
+		(lib_id "sierra-to-usb:Q_NMOS_TDSON_PQFN")
 		(at 450 120 0)
 		(unit 1)
@@
 		(property "Distributor" "DigiKey" (at 450 120 0) (hide yes) (effects (font (size 1.27 1.27))))
 		(property "EP-VIA" "yes" (at 450 120 0) (hide yes) (effects (font (size 1.27 1.27))))
-		(pin "D"
-		)
-		(pin "G"
-		)
-		(pin "S"
+		(pin "5"
+		)
+		(pin "4"
+		)
+		(pin "1"
 		)
 		(instances
@@
 	)
 	(symbol
-		(lib_id "Device:Q_NPN")
+		(lib_id "sierra-to-usb:Q_NPN_SOT89")
 		(at 440 105 0)
 		(unit 1)
@@
 		(property "MPN" "Central Semi FCX493TA" (at 440 105 0) (hide yes) (effects (font (size 1.27 1.27))))
 		(property "Distributor" "LCSC" (at 440 105 0) (hide yes) (effects (font (size 1.27 1.27))))
-		(pin "B"
-		)
-		(pin "C"
-		)
-		(pin "E"
+		(pin "1"
+		)
+		(pin "2"
+		)
+		(pin "3"
 		)
 		(instances
@@
 	)
 	(symbol
-		(lib_id "Device:Q_NMOS")
+		(lib_id "sierra-to-usb:Q_NMOS_TDSON_PQFN")
 		(at 480 100 0)
 		(unit 1)
@@
 		(property "Distributor" "DigiKey" (at 480 100 0) (hide yes) (effects (font (size 1.27 1.27))))
 		(property "EP-VIA" "yes" (at 480 100 0) (hide yes) (effects (font (size 1.27 1.27))))
-		(pin "D"
-		)
-		(pin "G"
-		)
-		(pin "S"
+		(pin "5"
+		)
+		(pin "4"
+		)
+		(pin "1"
 		)
 		(instances
@@
 	)
 	(symbol
-		(lib_id "Device:Q_NPN")
+		(lib_id "sierra-to-usb:Q_NPN_SOT89")
 		(at 470 115 0)
 		(unit 1)
@@
 		(property "MPN" "Central Semi FCX493TA" (at 470 115 0) (hide yes) (effects (font (size 1.27 1.27))))
 		(property "Distributor" "LCSC" (at 470 115 0) (hide yes) (effects (font (size 1.27 1.27))))
-		(pin "B"
-		)
-		(pin "C"
-		)
-		(pin "E"
+		(pin "1"
+		)
+		(pin "2"
+		)
+		(pin "3"
 		)
 		(instances
@@
 	)
 	(symbol
-		(lib_id "Device:Q_NMOS")
+		(lib_id "sierra-to-usb:Q_NMOS_DPAK")
 		(at 600 30 0)
 		(unit 1)
@@
 		(property "MPN" "Infineon IRLR7843TRPBF" (at 600 30 0) (hide yes) (effects (font (size 1.27 1.27))))
 		(property "Distributor" "DigiKey" (at 600 30 0) (hide yes) (effects (font (size 1.27 1.27))))
-		(pin "D"
-		)
-		(pin "G"
-		)
-		(pin "S"
+		(pin "2"
+		)
+		(pin "1"
+		)
+		(pin "3"
 		)
 		(instances
@@
 	)
 	(symbol
-		(lib_id "Device:Q_NMOS")
+		(lib_id "sierra-to-usb:Q_NMOS_DPAK")
 		(at 600 60 0)
 		(unit 1)
@@
 		(property "MPN" "Infineon IRLR7843TRPBF" (at 600 60 0) (hide yes) (effects (font (size 1.27 1.27))))
 		(property "Distributor" "DigiKey" (at 600 60 0) (hide yes) (effects (font (size 1.27 1.27))))
-		(pin "D"
-		)
-		(pin "G"
-		)
-		(pin "S"
-		)
-		(instances
+		(pin "2"
+		)
+		(pin "1"
+		)
+		(pin "3"
+		)
+		(instances
