File: full-adapter/cad/processor-control.kicad_sch (KiCad schematic)
At the start: 8 parts, among them U1 RK3568B2

Commit message: Capture power-off-isolated Linux debug console with verified connector
Other:
- note added: "I2C0 connects both RK809 and RK860. 1.8V pull-ups and PMIC series resistors are on the PMIC page. See console page for isolated 3.3V adapter interface."
- note removed: "I2C0 connects both RK809 and RK860. 1.8V pull-ups and PMIC series resistors are on the PMIC page. Console connector/level conversion remain to be captured."
Changed lines of the file:
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@@
 (property "Description" "Power symbol creates a global label with name \"GND\" , ground" (at 137.16 213.36 0) (effects (font (size 1.27 1.27))) (hide yes))
 (pin "1")(instances (project "full-adapter" (path "/fda20879-fa66-56c0-be14-de2506349b46/0a3d8b6b-806a-5303-a7dc-3b535bf2187e" (reference "#PWRprocessorcontrol001") (unit 1)))))
-(text "I2C0 connects both RK809 and RK860.\n1.8V pull-ups and PMIC series resistors are on the PMIC page.\nConsole connector/level conversion remain to be captured." (at 17.78 208.28 0) (effects (font (size 1.1 1.1)) (justify left top)))
+(text "I2C0 connects both RK809 and RK860.\n1.8V pull-ups and PMIC series resistors are on the PMIC page.\nSee console page for isolated 3.3V adapter interface." (at 17.78 208.28 0) (effects (font (size 1.1 1.1)) (justify left top)))
 (rectangle (start 198.12 15.24) (end 406.4 106.67999999999999) (stroke (width 0.254) (type default) (color 60 110 145 1)) (fill (type none)))
 (text "Hardware boot configuration" (at 201.93 19.05 0) (effects (font (size 1.8 1.8)) (justify left top)))
