File: full-adapter/cad/ethernet-pcie.kicad_sch (KiCad schematic)
At the start: 11 parts, among them U1 RK3568B2, U11 RTL8125BG-CG

Commit message: Capture PCIe control isolation and Ethernet startup reset
Other:
- note added: "Control pull-ups use the Ethernet supply. U14 isolates WAKE/CLKREQ; U16 delays reset release. Fast power-loss timing remains open."
- note added: "Reference clock outputs to the endpoint in RC mode. MULTI_PHY2 is dedicated to PCIe2; do not select SATA2/QSGMII. Functional CLKREQn/WAKEn M1 on VCCIO5 are on the control page."
- note added: "U16 releases PERSTB after its hardware delay; R679 retains a local pulldown. Control rails remain isolated by U14/U15. Route each lane as a controlled-impedance pair with no stubs. C687/C688 at U1; C689/C690 at U11. Full routing and signal validation remain open."
- note removed: "Control pull-ups use the Ethernet supply. Host-side isolation, reset qualification and functional GPIO connections are unfinished."
- note removed: "R679 holds PERSTB asserted until the hardware reset circuit is added. Do not bridge control pins directly across the two 3.3V domains. Route each lane as a controlled-impedance pair with no stubs. C687/C688 at U1; C689/C690 at U11. Full routing and signal validation remain open."
- note removed: "Reference clock outputs to the endpoint in RC mode. MULTI_PHY2 is dedicated to PCIe2; do not select SATA2/QSGMII. Select functional CLKREQn/WAKEn M1 on VCCIO5 later."
Changed lines of the file:
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@@
 (wire (pts (xy 111.76 73.66) (xy 119.38 73.66)) (stroke (width 0) (type default)))
 (label "PCIE_REFCLK_N" (at 119.38 73.66 0)  (effects (font (size 1.27 1.27)) (justify left bottom)))
-(text "Reference clock outputs to the endpoint in RC mode.\nMULTI_PHY2 is dedicated to PCIe2; do not select SATA2/QSGMII.\nSelect functional CLKREQn/WAKEn M1 on VCCIO5 later." (at 17.78 101.6 0) (effects (font (size 1.05 1.05)) (justify left top)))
+(text "Reference clock outputs to the endpoint in RC mode.\nMULTI_PHY2 is dedicated to PCIe2; do not select SATA2/QSGMII.\nFunctional CLKREQn/WAKEn M1 on VCCIO5 are on the control page." (at 17.78 101.6 0) (effects (font (size 1.05 1.05)) (justify left top)))
 (rectangle (start 215.9 15.24) (end 406.4 121.92) (stroke (width 0.254) (type default) (color 60 110 145 1)) (fill (type none)))
 (text "RTL8125BG PCIe endpoint" (at 219.71 19.05 0) (effects (font (size 1.8 1.8)) (justify left top)))
@@
 (label "ETH_ISOLATE_N" (at 287.02 60.96 180)  (effects (font (size 1.27 1.27)) (justify right bottom)))
 (wire (pts (xy 330.2 60.96) (xy 337.82 60.96)) (stroke (width 0) (type default)))
-(label "ETH_WAKE_N" (at 337.82 60.96 0)  (effects (font (size 1.27 1.27)) (justify left bottom)))
+(global_label "ETH_WAKE_N" (at 337.82 60.96 0) (shape bidirectional) (effects (font (size 1.27 1.27)) (justify left)))
 (wire (pts (xy 294.64 66.04) (xy 287.02 66.04)) (stroke (width 0) (type default)))
-(label "ETH_PERST_N" (at 287.02 66.04 180)  (effects (font (size 1.27 1.27)) (justify right bottom)))
+(global_label "ETH_PERST_N" (at 287.02 66.04 180) (shape bidirectional) (effects (font (size 1.27 1.27)) (justify right)))
 (wire (pts (xy 330.2 66.04) (xy 337.82 66.04)) (stroke (width 0) (type default)))
 (label "ETH_PCIE_TX_P" (at 337.82 66.04 0)  (effects (font (size 1.27 1.27)) (justify left bottom)))
@@
 (label "PCIE_REFCLK_N" (at 287.02 86.36 180)  (effects (font (size 1.27 1.27)) (justify right bottom)))
 (wire (pts (xy 294.64 91.44) (xy 287.02 91.44)) (stroke (width 0) (type default)))
-(label "ETH_CLKREQ_N" (at 287.02 91.44 180)  (effects (font (size 1.27 1.27)) (justify right bottom)))
-(text "Control pull-ups use the Ethernet supply. Host-side isolation,\nreset qualification and functional GPIO connections are unfinished." (at 223.52 109.22 0) (effects (font (size 1.05 1.05)) (justify left top)))
+(global_label "ETH_CLKREQ_N" (at 287.02 91.44 180) (shape bidirectional) (effects (font (size 1.27 1.27)) (justify right)))
+(text "Control pull-ups use the Ethernet supply. U14 isolates WAKE/CLKREQ;\nU16 delays reset release. Fast power-loss timing remains open." (at 223.52 109.22 0) (effects (font (size 1.05 1.05)) (justify left top)))
 (rectangle (start 10.16 129.54) (end 406.40000000000003 185.42) (stroke (width 0.254) (type default) (color 60 110 145 1)) (fill (type none)))
 (text "One AC capacitor per transmit leg — at its source" (at 13.97 133.35 0) (effects (font (size 1.8 1.8)) (justify left top)))
@@
 (pin "1")(instances (project "full-adapter" (path "/fda20879-fa66-56c0-be14-de2506349b46/3d4110a4-f8aa-5e5b-a063-38d346e79b21" (reference "#PWRethernetpcie001") (unit 1)))))
 (wire (pts (xy 38.1 220.98) (xy 38.1 231.14)) (stroke (width 0) (type default)))
-(label "ETH_WAKE_N" (at 38.1 231.14 0)  (effects (font (size 1.27 1.27)) (justify left bottom)))
+(global_label "ETH_WAKE_N" (at 38.1 231.14 0) (shape bidirectional) (effects (font (size 1.27 1.27)) (justify left)))
 (symbol (lib_id "Device:R_Small_US") (at 116.84 218.44 0) (unit 1) (in_bom yes) (on_board yes) (dnp no) (property "Reference" "R678" (at 119.38000000000001 217.17 0) (effects (font (size 1.27 1.27)) (justify left)))
 (property "Value" "4.7kR 1%" (at 119.38000000000001 219.70999999999998 0) (effects (font (size 1.27 1.27)) (justify left)))
@@
 (pin "1")(instances (project "full-adapter" (path "/fda20879-fa66-56c0-be14-de2506349b46/3d4110a4-f8aa-5e5b-a063-38d346e79b21" (reference "#PWRethernetpcie002") (unit 1)))))
 (wire (pts (xy 116.84 220.98) (xy 116.84 231.14)) (stroke (width 0) (type default)))
-(label "ETH_CLKREQ_N" (at 116.84 231.14 0)  (effects (font (size 1.27 1.27)) (justify left bottom)))
+(global_label "ETH_CLKREQ_N" (at 116.84 231.14 0) (shape bidirectional) (effects (font (size 1.27 1.27)) (justify left)))
 (symbol (lib_id "Device:R_Small_US") (at 198.12 228.6 0) (unit 1) (in_bom yes) (on_board yes) (dnp no) (property "Reference" "R679" (at 200.66 227.32999999999998 0) (effects (font (size 1.27 1.27)) (justify left)))
 (property "Value" "47kR 1%" (at 200.66 229.86999999999998 0) (effects (font (size 1.27 1.27)) (justify left)))
@@
 (pin "2")(instances (project "full-adapter" (path "/fda20879-fa66-56c0-be14-de2506349b46/3d4110a4-f8aa-5e5b-a063-38d346e79b21" (reference "R679") (unit 1)))))
 (wire (pts (xy 198.12 226.06) (xy 198.12 213.36)) (stroke (width 0) (type default)))
-(label "ETH_PERST_N" (at 198.12 213.36 0)  (effects (font (size 1.27 1.27)) (justify left bottom)))
+(global_label "ETH_PERST_N" (at 198.12 213.36 0) (shape bidirectional) (effects (font (size 1.27 1.27)) (justify left)))
 (wire (pts (xy 198.12 231.14) (xy 198.12 238.76)) (stroke (width 0) (type default)))
 (symbol (lib_id "power:GND") (at 198.12 238.76 0) (unit 1) (in_bom no) (on_board no) (dnp no) (property "Reference" "#PWRethernetpcie003" (at 198.12 243.84 0) (effects (font (size 1.27 1.27))) (hide yes))
@@
 (property "Description" "Power symbol creates a global label with name \"GND\" , ground" (at 353.06 243.84 0) (effects (font (size 1.27 1.27))) (hide yes))
 (pin "1")(instances (project "full-adapter" (path "/fda20879-fa66-56c0-be14-de2506349b46/3d4110a4-f8aa-5e5b-a063-38d346e79b21" (reference "#PWRethernetpcie005") (unit 1)))))
-(text "R679 holds PERSTB asserted until the hardware reset circuit is added. Do not bridge control pins directly across the two 3.3V domains.\nRoute each lane as a controlled-impedance pair with no stubs. C687/C688 at U1; C689/C690 at U11. Full routing and signal validation remain open." (at 15.24 266.7 0) (effects (font (size 1.05 1.05)) (justify left top)))
+(text "U16 releases PERSTB after its hardware delay; R679 retains a local pulldown. Control rails remain isolated by U14/U15.\nRoute each lane as a controlled-impedance pair with no stubs. C687/C688 at U1; C689/C690 at U11. Full routing and signal validation remain open." (at 15.24 266.7 0) (effects (font (size 1.05 1.05)) (justify left top)))
 )
