File: full-adapter/cm4/cad/cm4-interfaces.kicad_sch (KiCad schematic)
At the start: 2 parts, among them J100 DF40C-100DS-0.4V(58), J101 DF40C-100DS-0.4V(58)

Commit message: Capture CM4 gigabit magnetics and isolated PoE termination
Other:
- note added: "Four MDI pairs connect to T120 on ethernet-data. PoE extraction stays on the isolated cable side. No discrete external Ethernet PHY or PCIe NIC. SYNC and LED contacts currently unused."
- note added: "Native gigabit PHY / HX6096NL magnetics"
- note removed: "Four MDI pairs require qualified 1:1 gigabit magnetics. PoE extraction stays on the isolated cable side. No discrete external Ethernet PHY or PCIe NIC. SYNC and LED contacts currently unused."
- note removed: "Native gigabit PHY / magnetics integration pending"
Changed lines of the file:
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@@
 (title_block (title "CM4 Lite: native gigabit and PCIe USB3 host interfaces") (rev "WORK IN PROGRESS") (company "Integrated modem development board"))
 (rectangle (start 10.16 15.24) (end 200.66 231.14000000000001) (stroke (width 0.254) (type default) (color 60 110 145 1)) (fill (type none)))
-(text "Native gigabit PHY / magnetics integration pending" (at 13.97 19.05 0) (effects (font (size 1.8 1.8)) (justify left top)))
+(text "Native gigabit PHY / HX6096NL magnetics" (at 13.97 19.05 0) (effects (font (size 1.8 1.8)) (justify left top)))
 (symbol (lib_id "cm4:CM4_J1") (at 93.98 78.74 0) (unit 4) (in_bom yes) (on_board yes) (dnp no) (property "Reference" "J100" (at 93.98 50.8 0) (effects (font (size 1.27 1.27))))
 (property "Value" "DF40C-100DS-0.4V(58)" (at 93.98 53.339999999999996 0) (effects (font (size 1.27 1.27))))
@@
 (no_connect (at 121.92 88.9))
 (no_connect (at 121.92 91.44))
-(text "Four MDI pairs require qualified 1:1 gigabit magnetics.\nPoE extraction stays on the isolated cable side.\nNo discrete external Ethernet PHY or PCIe NIC.\nSYNC and LED contacts currently unused." (at 17.78 144.78 0) (effects (font (size 1.27 1.27)) (justify left top)))
+(text "Four MDI pairs connect to T120 on ethernet-data.\nPoE extraction stays on the isolated cable side.\nNo discrete external Ethernet PHY or PCIe NIC.\nSYNC and LED contacts currently unused." (at 17.78 144.78 0) (effects (font (size 1.27 1.27)) (justify left top)))
 (rectangle (start 213.36 15.24) (end 403.86 231.14000000000001) (stroke (width 0.254) (type default) (color 60 110 145 1)) (fill (type none)))
 (text "PCIe Gen2 x1 to dedicated USB3 host / USB2 recovery" (at 217.17000000000002 19.05 0) (effects (font (size 1.8 1.8)) (justify left top)))
