File: hardware/supervisor.kicad_sch (KiCad schematic)
At the start: 14 parts, among them J201 SWD / recovery, J202 WDT RUN jumper, SW201 RESET, U201 STM32G0B1CCT6, U202 TPS3823-33DBVR

Commit message: Prepare audited RK3566 pin table and resolve recovery resistors and headers
Parts:
- J201: footprint Connector_PinHeader_2.54mm:PinHeader_1x06_P2.54mm_Vertical -> Recovery:Wuerth_61300611121_1x06_P2.54mm_Vertical; MPN (none) -> 61300611121; Manufacturer (none) -> Wuerth Elektronik
- J202: footprint Connector_PinHeader_2.54mm:PinHeader_1x02_P2.54mm_Vertical -> Recovery:Wuerth_61300211121_1x02_P2.54mm_Vertical; MPN (none) -> 61300211121; Manufacturer (none) -> Wuerth Elektronik; Required Mating Part (none) -> 60900213421; fit RUN shunt for unattended operation
- R201, R202, R203: LCSC (none) -> C98220; MPN (none) -> RC0603FR-0710KL; Manufacturer (none) -> Yageo; Power Rating (none) -> 0.1W; Tolerance (none) -> 1%; Voltage Rating (none) -> 75V

Commit message: Resolve recovery reset switch against manufacturer drawing
Parts:
- SW201: Contact Rating (none) -> 12VDC 50mA; LCSC (none) -> C2886898; MPN (none) -> TL3342F160QG; Manufacturer (none) -> E-Switch; Operating Temperature (none) -> -20 to +70 C
Changed lines of the file:
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@@
   (symbol (lib_id "power:GND") (at 218.44 185.42 0) (unit 1) (in_bom no) (on_board yes) (dnp no) (property "Reference" "#PWR137" (at 222.25 182.88 0) (effects (font (size 1.27 1.27)) (justify left) (hide yes))) (property "Value" "GND" (at 219.71 189.23 0) (effects (font (size 1.27 1.27)) (justify left))) (property "Footprint" "" (at 218.44 185.42 0) (effects (font (size 1.27 1.27)) (justify left) (hide yes))) (property "Datasheet" "" (at 218.44 185.42 0) (effects (font (size 1.27 1.27)) (justify left) (hide yes))) (pin "1") (instances (project "recovery" (path "/37b14702-5d54-5543-b96e-899c36eac351/3d1f41aa-40e8-59ac-82e1-1b8621dcb8ce" (reference "#PWR137") (unit 1)))))
   (text "VTref only; debugger must not power the target.\nLeave debug unlocked until signed-update recovery is proven.\nNo USB data path through this MCU." (at 218.44 199.39 0) (effects (font (size 1.27 1.27)) (justify left)))
-  (symbol (lib_id "Switch:SW_Push") (at 335.28 165.1 0) (unit 1) (in_bom yes) (on_board yes) (dnp no) (property "Reference" "SW201" (at 330.2 157.48 0) (effects (font (size 1.27 1.27)) (justify left))) (property "Value" "RESET" (at 330.2 160.02 0) (effects (font (size 1.27 1.27)) (justify left))) (property "Footprint" "Button_Switch_SMD:SW_SPST_TL3342" (at 335.28 165.1 0) (effects (font (size 1.27 1.27)) (justify left) (hide yes))) (property "Datasheet" "" (at 335.28 165.1 0) (effects (font (size 1.27 1.27)) (justify left) (hide yes))) (pin "1") (pin "2") (instances (project "recovery" (path "/37b14702-5d54-5543-b96e-899c36eac351/3d1f41aa-40e8-59ac-82e1-1b8621dcb8ce" (reference "SW201") (unit 1)))))
+  (symbol (lib_id "Switch:SW_Push") (at 335.28 165.1 0) (unit 1) (in_bom yes) (on_board yes) (dnp no) (property "Reference" "SW201" (at 330.2 157.48 0) (effects (font (size 1.27 1.27)) (justify left))) (property "Value" "RESET" (at 330.2 160.02 0) (effects (font (size 1.27 1.27)) (justify left))) (property "Footprint" "Button_Switch_SMD:SW_SPST_TL3342" (at 335.28 165.1 0) (effects (font (size 1.27 1.27)) (justify left) (hide yes))) (property "Datasheet" "https://configured-product-images.s3.amazonaws.com/2D/specs/TL3342F160QG.pdf" (at 335.28 165.1 0) (effects (font (size 1.27 1.27)) (hide yes))) (pin "1") (pin "2") (instances (project "recovery" (path "/37b14702-5d54-5543-b96e-899c36eac351/3d1f41aa-40e8-59ac-82e1-1b8621dcb8ce" (reference "SW201") (unit 1)))) (property "MPN" "TL3342F160QG" (at 335.28 165.1 0) (effects (font (size 1.27 1.27)) (hide yes))) (property "Manufacturer" "E-Switch" (at 335.28 165.1 0) (effects (font (size 1.27 1.27)) (hide yes))) (property "LCSC" "C2886898" (at 335.28 165.1 0) (effects (font (size 1.27 1.27)) (hide yes))) (property "Contact Rating" "12VDC 50mA" (at 335.28 165.1 0) (effects (font (size 1.27 1.27)) (hide yes))) (property "Operating Temperature" "-20 to +70 C" (at 335.28 165.1 0) (effects (font (size 1.27 1.27)) (hide yes))))
   (wire (pts (xy 330.2 165.1) (xy 322.58 165.1)) (stroke (width 0) (type default)))
   (label "MANUAL_RESET_N" (at 322.58 165.1 0) (effects (font (size 1.27 1.27)) (justify right bottom)))

Commit message: Select recovery bypass capacitors and archive manufacturer bias curves
Parts:
- C201, C202: DC Bias Review (none) -> Typical +0.94% at 3.3V, 25C; not guaranteed corner data; LCSC (none) -> C1590; MPN (none) -> CL10B104KA8NNNC; Manufacturer (none) -> Samsung Electro-Mechanics; Rating 16V X7R; verify DC-bias effective capacitance -> 25V X7R +/-10%; 0603
- C204, C205: DC Bias Review (none) -> Typical +0.94% at 3.3V, 25C; not guaranteed corner data; LCSC (none) -> C1590; MPN (none) -> CL10B104KA8NNNC; Manufacturer (none) -> Samsung Electro-Mechanics; Rating (none) -> 25V X7R +/-10%; 0603

Commit message: Capture provisional recovery bulk capacitor and MCU acceptance limits
Parts:
- C203: footprint Capacitor_SMD:C_0603_1608Metric -> Capacitor_SMD:C_0805_2012Metric; LCSC (none) -> C98195; MPN (none) -> CL21B475KAFNNNE; Manufacturer (none) -> Samsung Electro-Mechanics; Rating 16V X7R; verify DC-bias effective capacitance -> 25V X7R +/-10%; bias review pending; Selection Status (none) -> Provisional; about 4.08uF typical at 3.3V, before tolerance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
Changed lines of the file:
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@@
   (wire (pts (xy 154.94 68.58) (xy 154.94 76.2)) (stroke (width 0) (type default)))
   (junction (at 154.94 55.88) (diameter 0) (color 0 0 0 0))
-  (symbol (lib_id "Device:C_Small") (at 170.18 66.04 0) (unit 1) (in_bom yes) (on_board yes) (dnp no) (property "Reference" "C203" (at 173.99 63.50000000000001 0) (effects (font (size 1.27 1.27)) (justify left))) (property "Value" "4.7uF" (at 173.99 66.04 0) (effects (font (size 1.27 1.27)) (justify left))) (property "Footprint" "Capacitor_SMD:C_0603_1608Metric" (at 170.18 66.04 0) (effects (font (size 1.27 1.27)) (justify left) (hide yes))) (property "Datasheet" "" (at 170.18 66.04 0) (effects (font (size 1.27 1.27)) (justify left) (hide yes))) (property "Rating" "16V X7R; verify DC-bias effective capacitance" (at 170.18 66.04 0) (effects (font (size 1.27 1.27)) (hide yes))) (pin "1") (pin "2") (instances (project "recovery" (path "/37b14702-5d54-5543-b96e-899c36eac351/3d1f41aa-40e8-59ac-82e1-1b8621dcb8ce" (reference "C203") (unit 1)))))
+  (symbol (lib_id "Device:C_Small") (at 170.18 66.04 0) (unit 1) (in_bom yes) (on_board yes) (dnp no) (property "Reference" "C203" (at 173.99 63.50000000000001 0) (effects (font (size 1.27 1.27)) (justify left))) (property "Value" "4.7uF" (at 173.99 66.04 0) (effects (font (size 1.27 1.27)) (justify left))) (property "Footprint" "Capacitor_SMD:C_0805_2012Metric" (at 170.18 66.04 0) (effects (font (size 1.27 1.27)) (justify left) (hide yes))) (property "Datasheet" "https://product.samsungsem.com/mlcc/CL21B475KAFNNN.do" (at 170.18 66.04 0) (effects (font (size 1.27 1.27)) (justify left) (hide yes))) (property "Rating" "25V X7R +/-10%; bias review pending" (at 170.18 66.04 0) (effects (font (size 1.27 1.27)) (hide yes))) (pin "1") (pin "2") (instances (project "recovery" (path "/37b14702-5d54-5543-b96e-899c36eac351/3d1f41aa-40e8-59ac-82e1-1b8621dcb8ce" (reference "C203") (unit 1)))) (property "MPN" "CL21B475KAFNNNE" (at 170.18 66.04 0) (effects (font (size 1.27 1.27)) (hide yes))) (property "Manufacturer" "Samsung Electro-Mechanics" (at 170.18 66.04 0) (effects (font (size 1.27 1.27)) (hide yes))) (property "LCSC" "C98195" (at 170.18 66.04 0) (effects (font (size 1.27 1.27)) (hide yes))) (property "Selection Status" "Provisional; about 4.08uF typical at 3.3V, before tolerance/temp/aging" (at 170.18 66.04 0) (effects (font (size 1.27 1.27)) (hide yes))))
   (wire (pts (xy 170.18 63.5) (xy 170.18 55.88)) (stroke (width 0) (type default)))
   (wire (pts (xy 170.18 68.58) (xy 170.18 76.2)) (stroke (width 0) (type default)))

Commit message: Increase recovery bulk capacitance with documented bias margin
Parts:
- C203: value 4.7uF -> 10uF; footprint Capacitor_SMD:C_0805_2012Metric -> Capacitor_SMD:C_1206_3216Metric; LCSC C98195 -> C14860; MPN CL21B475KAFNNNE -> CL31B106KAHNNNE; Rating 25V X7R +/-10%; bias review pending -> 25V X7R +/-10%; bias margin reviewed; aging qualification p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; Selection Status Provisional; about 4.08uF typical at 3.3V, before tolerance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 -> 10uF selected for bias margin; typical combined estimate 6.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
Changed lines of the file:
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@@
   (wire (pts (xy 154.94 68.58) (xy 154.94 76.2)) (stroke (width 0) (type default)))
   (junction (at 154.94 55.88) (diameter 0) (color 0 0 0 0))
-  (symbol (lib_id "Device:C_Small") (at 170.18 66.04 0) (unit 1) (in_bom yes) (on_board yes) (dnp no) (property "Reference" "C203" (at 173.99 63.50000000000001 0) (effects (font (size 1.27 1.27)) (justify left))) (property "Value" "4.7uF" (at 173.99 66.04 0) (effects (font (size 1.27 1.27)) (justify left))) (property "Footprint" "Capacitor_SMD:C_0805_2012Metric" (at 170.18 66.04 0) (effects (font (size 1.27 1.27)) (justify left) (hide yes))) (property "Datasheet" "https://product.samsungsem.com/mlcc/CL21B475KAFNNN.do" (at 170.18 66.04 0) (effects (font (size 1.27 1.27)) (justify left) (hide yes))) (property "Rating" "25V X7R +/-10%; bias review pending" (at 170.18 66.04 0) (effects (font (size 1.27 1.27)) (hide yes))) (pin "1") (pin "2") (instances (project "recovery" (path "/37b14702-5d54-5543-b96e-899c36eac351/3d1f41aa-40e8-59ac-82e1-1b8621dcb8ce" (reference "C203") (unit 1)))) (property "MPN" "CL21B475KAFNNNE" (at 170.18 66.04 0) (effects (font (size 1.27 1.27)) (hide yes))) (property "Manufacturer" "Samsung Electro-Mechanics" (at 170.18 66.04 0) (effects (font (size 1.27 1.27)) (hide yes))) (property "LCSC" "C98195" (at 170.18 66.04 0) (effects (font (size 1.27 1.27)) (hide yes))) (property "Selection Status" "Provisional; about 4.08uF typical at 3.3V, before tolerance/temp/aging" (at 170.18 66.04 0) (effects (font (size 1.27 1.27)) (hide yes))))
+  (symbol (lib_id "Device:C_Small") (at 170.18 66.04 0) (unit 1) (in_bom yes) (on_board yes) (dnp no) (property "Reference" "C203" (at 173.99 63.50000000000001 0) (effects (font (size 1.27 1.27)) (justify left))) (property "Value" "10uF" (at 173.99 66.04 0) (effects (font (size 1.27 1.27)) (justify left))) (property "Footprint" "Capacitor_SMD:C_1206_3216Metric" (at 170.18 66.04 0) (effects (font (size 1.27 1.27)) (justify left) (hide yes))) (property "Datasheet" "https://product.samsungsem.com/mlcc/CL31B106KAHNNN.do" (at 170.18 66.04 0) (effects (font (size 1.27 1.27)) (justify left) (hide yes))) (property "Rating" "25V X7R +/-10%; bias margin reviewed; aging qualification pending" (at 170.18 66.04 0) (effects (font (size 1.27 1.27)) (hide yes))) (pin "1") (pin "2") (instances (project "recovery" (path "/37b14702-5d54-5543-b96e-899c36eac351/3d1f41aa-40e8-59ac-82e1-1b8621dcb8ce" (reference "C203") (unit 1)))) (property "MPN" "CL31B106KAHNNNE" (at 170.18 66.04 0) (effects (font (size 1.27 1.27)) (hide yes))) (property "Manufacturer" "Samsung Electro-Mechanics" (at 170.18 66.04 0) (effects (font (size 1.27 1.27)) (hide yes))) (property "LCSC" "C14860" (at 170.18 66.04 0) (effects (font (size 1.27 1.27)) (hide yes))) (property "Selection Status" "10uF selected for bias margin; typical combined estimate 6.48uF at 3.6V, -10% tolerance, -15% temperature; aging not included" (at 170.18 66.04 0) (effects (font (size 1.27 1.27)) (hide yes))))
   (wire (pts (xy 170.18 63.5) (xy 170.18 55.88)) (stroke (width 0) (type default)))
   (wire (pts (xy 170.18 68.58) (xy 170.18 76.2)) (stroke (width 0) (type default)))

Commit message: Connect open-drain watchdog directly to recovery MCU reset
Parts:
- removed D201: BAT54WS-7-F, Diode_SMD:D_SOD-323, symbol Device:D_Schottky_Small
- U202: value TPS3823-33DBVR -> TPS3828-33DBVR; symbol Power_Supervisor:TPS3823-xxDBV -> Recovery:TPS3828-xxDBV; LCSC C7719 -> C20032; MPN TPS3823-33DBVR -> TPS3828-33DBVR
Connections:
- net WDT_RESET_N is gone; now on net MCU_NRST_N: U202.1 (~{RESET})
Other:
- note added: "1.6s nominal watchdog; 2.93V threshold; 200ms nominal reset. Open-drain RESET directly shares MCU NRST with SWD. Verify NRST low-voltage margin across temperature before release."
- note added: "100nF at VDD/VREF; 10uF local bulk. No external clock required for UART/GPIO supervision."
- note removed: "1.6s nominal watchdog; 2.93V threshold; 200ms nominal reset. D201 isolates push-pull reset from SWD/manual NRST assertion. Verify NRST low-voltage margin across temperature before release."
- note removed: "100nF at VDD/VREF; 4.7uF local bulk. No external clock required for UART/GPIO supervision."
