File: hardware/always-on.kicad_sch (KiCad schematic)
At the start: 5 parts, among them U401 TPS62177DQCR

Commit message: Prepare audited RK3566 pin table and resolve recovery resistors and headers
Parts:
- R401: LCSC (none) -> C14675; Power Rating (none) -> 0.1W; Tolerance (none) -> 1%

Commit message: Increase always-on input capacitance for DC-bias margin
Parts:
- C401: value 2.2uF / 50V -> 4.7uF / 50V; LCSC C50254 -> C51205; MPN CL31B225KBHNNNE -> CL31B475KBHNNNE

Commit message: Add parallel always-on output capacitor with explicit stability gate
Parts:
- added C403: 22uF / 25V, Capacitor_SMD:C_1210_3225Metric, symbol Device:C_Small
Connections:
- net +3V3: now also C403.1
- net GND: now also C403.2
Other:
- note added: "TI SLVSB35C, Figure 8 / Tables 2-3. 10uH + 2x22uF nominal. Capacitor DC bias, complete rail load and layout review remain open. Route VOS as Kelvin sense after L401; join AGND / PGND / exposed pad locally."
- note removed: "TI SLVSB35C, Figure 8 / Tables 2-3. 10uH + 22uF nominal. Capacitor DC bias, complete rail load and layout review remain open. Route VOS as Kelvin sense after L401; join AGND / PGND / exposed pad locally."
