File: hardware/phy-power.kicad_sch (KiCad schematic)
At the start: 4 parts

Commit message: Complete appliance engineering schematic capture
Other:
- note added: "USB ANALOG FILTERS: local pin bypass and processor loads are captured. 45mOhm maximum DCR differs from 30mOhm reference example. Rail headroom, thermal limits and bead/capacitor damping remain to verify."
- note removed: "DRAFT USB ANALOG FILTERS: local pin bypass and processor loads still required. 45mOhm maximum DCR differs from 30mOhm reference example. Rail headroom, thermal limits and bead/capacitor damping remain to verify."
- title: USB PHY analog filters — DRAFT -> USB PHY analog filters — engineering capture
