File: hardware/poe-flyback.kicad_sch (KiCad schematic)
At the start: 78 parts, among them J1711 ED555/2DS, J1712 87898-0204, Q1705 150V, Q1707 20 V, T1702 30uH, U1702 LM51551QDSSRQ1, U1703 FOD817AS, U1704 TL431LIAIDBZR

Commit message: Audit appliance footprints, models and native schematic PCB synchronization
Parts:
- C1720: footprint PoE:TI_1812_254_1 -> Capacitor_SMD:C_1812_4532Metric_Pad1.57x3.40mm_HandSolder
- C1721, C1726, C1731, C1732, C1740: footprint PoE:TI_0805_HV -> Capacitor_SMD:C_0805_2012Metric_Pad1.18x1.45mm_HandSolder
- C1722, C1723, C1724, C1725: footprint PoE:TI_1210_270 -> Capacitor_SMD:C_1210_3225Metric_Pad1.33x2.70mm_HandSolder
- C1728, C1729, C1730: footprint PoE:TI_1210_280 -> Capacitor_SMD:C_1210_3225Metric_Pad1.33x2.70mm_HandSolder
- C1733, C1738: footprint PoE:TI_0603L -> Capacitor_SMD:C_0603_1608Metric_Pad1.08x0.95mm_HandSolder
- C1734, C1737: footprint PoE:TI_0603_1 -> Capacitor_SMD:C_0603_1608Metric_Pad1.08x0.95mm_HandSolder
- C1735, C1744, C1745: footprint PoE:TI_0603L_1 -> Capacitor_SMD:C_0603_1608Metric_Pad1.08x0.95mm_HandSolder
- C1736: footprint PoE:TI_1812_254 -> Capacitor_SMD:C_1812_4532Metric_Pad1.57x3.40mm_HandSolder
- C1739: footprint PoE:TI_0603_3 -> Capacitor_SMD:C_0603_1608Metric_Pad1.08x0.95mm_HandSolder
- C1741, C1743: footprint PoE:TI_0603 -> Capacitor_SMD:C_0603_1608Metric_Pad1.08x0.95mm_HandSolder
- C1746: footprint PoE:TI_0805L -> Capacitor_SMD:C_0805_2012Metric_Pad1.18x1.45mm_HandSolder
- D1714: footprint PoE:TI_SMA -> Diode_SMD:D_SMA_Handsoldering
- D1715, D1717: footprint PoE:TI_SOD-123 -> Diode_SMD:D_SOD-123
- D1716: footprint PoE:TI_WL-SMCW_YELLOW -> LED_SMD:LED_0603_1608Metric_Pad1.05x0.95mm_HandSolder
- D1718: footprint PoE:TI_PowerDI5 -> Appliance:Diodes_PowerDI-5_3Pin_Derived
- D1719: footprint PoE:TI_SOD-123_1 -> Diode_SMD:D_SOD-123
- D1721: footprint PoE:TI_SOT-23 -> Package_TO_SOT_SMD:SOT-23_Handsoldering
- L1707: footprint PoE:TI_XFL4020 -> Inductor_SMD:L_Coilcraft_XxL4020
- L1708: footprint PoE:TI_XAL5030 -> Inductor_SMD:L_Coilcraft_XAL5030-XXX
- Q1707: footprint PoE:TI_SOT-23_1 -> Package_TO_SOT_SMD:SOT-23_Handsoldering
- R1733: footprint PoE:TI_1206 -> Resistor_SMD:R_1206_3216Metric_Pad1.30x1.75mm_HandSolder
- R1734, R1735, R1740, R1742, R1743, R1745, R1746, R1757: footprint PoE:TI_0603 -> Resistor_SMD:R_0603_1608Metric_Pad0.98x0.95mm_HandSolder
- R1736: footprint PoE:TI_2010L -> Resistor_SMD:R_2010_5025Metric_Pad1.40x2.65mm_HandSolder
- R1737, R1741, R1744, R1753, R1760, R1763: footprint PoE:TI_0603_2 -> Resistor_SMD:R_0603_1608Metric_Pad0.98x0.95mm_HandSolder
- R1738: footprint PoE:TI_2010 -> Resistor_SMD:R_2010_5025Metric_Pad1.40x2.65mm_HandSolder
- R1739: footprint PoE:TI_0805_HV_1 -> Resistor_SMD:R_0805_2012Metric_Pad1.20x1.40mm_HandSolder
- R1747, R1748: footprint PoE:TI_2512 -> Resistor_SMD:R_2512_6332Metric_Pad1.40x3.35mm_HandSolder
- R1754, R1762: footprint PoE:TI_0603L -> Resistor_SMD:R_0603_1608Metric_Pad0.98x0.95mm_HandSolder
- R1755, R1756, R1759, R1761: footprint PoE:TI_0603L_2 -> Resistor_SMD:R_0603_1608Metric_Pad0.98x0.95mm_HandSolder
- U1702: footprint PoE:TI_DSS0012C -> Package_SON:WSON-12-1EP_3x2mm_P0.5mm_EP1x2.65
- U1704: footprint PoE:TI_DBZ0003A_M -> Package_TO_SOT_SMD:SOT-23_Handsoldering
