File: hardware/poe-input.kicad_sch (KiCad schematic)
At the start: 30 parts, among them Q1701 100V, Q1702 100V, Q1703 100V, Q1704 100V

Commit message: Audit appliance footprints, models and native schematic PCB synchronization
Parts:
- C1707, C1708, C1709, C1710, C1711, C1712: footprint PoE:TI_0603_1 -> Capacitor_SMD:C_0603_1608Metric_Pad1.08x0.95mm_HandSolder
- D1701, D1702, D1703, D1704, D1706, D1707, D1708, D1709: footprint PoE:TI_SMB -> Diode_SMD:D_SMB_Handsoldering
- D1705: footprint PoE:TI_SMB_1 -> Diode_SMD:D_SMB_Handsoldering
- L1701, L1703: footprint PoE:TI_WE-CBF_0603 -> Inductor_SMD:L_0603_1608Metric_Pad1.05x0.95mm_HandSolder
- Q1701, Q1702, Q1703, Q1704: footprint PoE:TI_SSOT-3 -> Package_TO_SOT_SMD:SuperSOT-3
- R1709, R1710, R1711, R1712, R1713, R1714, R1715, R1716: footprint PoE:TI_0603_2 -> Resistor_SMD:R_0603_1608Metric_Pad0.98x0.95mm_HandSolder
Changed lines of the file:
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@@
 			)
 		)
-		(property "Footprint" "PoE:TI_WE-CBF_0603"
+		(property "Footprint" "Inductor_SMD:L_0603_1608Metric_Pad1.05x0.95mm_HandSolder"
 			(at 320.04 193.04 0)
 			(hide yes)
@@
 			)
 		)
-		(property "Footprint" "PoE:TI_0603_1"
+		(property "Footprint" "Capacitor_SMD:C_0603_1608Metric_Pad1.08x0.95mm_HandSolder"
 			(at 109.22 185.42 0)
 			(hide yes)
@@
 			)
 		)
-		(property "Footprint" "PoE:TI_0603_2"
+		(property "Footprint" "Resistor_SMD:R_0603_1608Metric_Pad0.98x0.95mm_HandSolder"
 			(at 119.38 185.42 0)
 			(hide yes)
@@
 			)
 		)
-		(property "Footprint" "PoE:TI_SSOT-3"
+		(property "Footprint" "Package_TO_SOT_SMD:SuperSOT-3"
 			(at 190.5 177.8 0)
 			(hide yes)
@@
 			)
 		)
-		(property "Footprint" "PoE:TI_0603_1"
+		(property "Footprint" "Capacitor_SMD:C_0603_1608Metric_Pad1.08x0.95mm_HandSolder"
 			(at 200.66 185.42 0)
 			(hide yes)
@@
 			)
 		)
-		(property "Footprint" "PoE:TI_SMB"
+		(property "Footprint" "Diode_SMD:D_SMB_Handsoldering"
 			(at 243.84 147.32 0)
 			(hide yes)
@@
 			)
 		)
-		(property "Footprint" "PoE:TI_SMB"
+		(property "Footprint" "Diode_SMD:D_SMB_Handsoldering"
 			(at 152.4 147.32 0)
 			(hide yes)
@@
 			)
 		)
-		(property "Footprint" "PoE:TI_0603_2"
+		(property "Footprint" "Resistor_SMD:R_0603_1608Metric_Pad0.98x0.95mm_HandSolder"
 			(at 210.82 185.42 0)
 			(hide yes)
@@
 			)
 		)
-		(property "Footprint" "PoE:TI_SMB"
+		(property "Footprint" "Diode_SMD:D_SMB_Handsoldering"
 			(at 175.26 175.26 0)
 			(hide yes)
@@
 			)
 		)
-		(property "Footprint" "PoE:TI_0603_1"
+		(property "Footprint" "Capacitor_SMD:C_0603_1608Metric_Pad1.08x0.95mm_HandSolder"
 			(at 139.7 185.42 0)
 			(hide yes)
@@
 			)
 		)
-		(property "Footprint" "PoE:TI_SSOT-3"
+		(property "Footprint" "Package_TO_SOT_SMD:SuperSOT-3"
 			(at 149.86 177.8 0)
 			(hide yes)
@@
 			)
 		)
-		(property "Footprint" "PoE:TI_0603_1"
+		(property "Footprint" "Capacitor_SMD:C_0603_1608Metric_Pad1.08x0.95mm_HandSolder"
 			(at 287.02 167.64 0)
 			(hide yes)
@@
 			)
 		)
-		(property "Footprint" "PoE:TI_SMB"
+		(property "Footprint" "Diode_SMD:D_SMB_Handsoldering"
 			(at 96.52 147.32 0)
 			(hide yes)
@@
 			)
 		)
-		(property "Footprint" "PoE:TI_0603_2"
+		(property "Footprint" "Resistor_SMD:R_0603_1608Metric_Pad0.98x0.95mm_HandSolder"
 			(at 210.82 170.18 0)
 			(hide yes)
@@
 			)
 		)
-		(property "Footprint" "PoE:TI_0603_2"
+		(property "Footprint" "Resistor_SMD:R_0603_1608Metric_Pad0.98x0.95mm_HandSolder"
 			(at 132.08 170.18 0)
 			(hide yes)
@@
 			)
 		)
-		(property "Footprint" "PoE:TI_SSOT-3"
+		(property "Footprint" "Package_TO_SOT_SMD:SuperSOT-3"
 			(at 99.06 177.8 0)
 			(hide yes)
@@
 			)
 		)
-		(property "Footprint" "PoE:TI_WE-CBF_0603"
+		(property "Footprint" "Inductor_SMD:L_0603_1608Metric_Pad1.05x0.95mm_HandSolder"
 			(at 320.04 139.7 0)
 			(hide yes)
@@
 			)
 		)
-		(property "Footprint" "PoE:TI_0603_2"
+		(property "Footprint" "Resistor_SMD:R_0603_1608Metric_Pad0.98x0.95mm_HandSolder"
 			(at 132.08 185.42 0)
 			(hide yes)
@@
 			)
 		)
-		(property "Footprint" "PoE:TI_0603_2"
+		(property "Footprint" "Resistor_SMD:R_0603_1608Metric_Pad0.98x0.95mm_HandSolder"
 			(at 223.52 185.42 0)
 			(hide yes)
@@
 			)
 		)
-		(property "Footprint" "PoE:TI_SMB"
+		(property "Footprint" "Diode_SMD:D_SMB_Handsoldering"
 			(at 187.96 147.32 0)
 			(hide yes)
@@
 			)
 		)
-		(property "Footprint" "PoE:TI_0603_1"
+		(property "Footprint" "Capacitor_SMD:C_0603_1608Metric_Pad1.08x0.95mm_HandSolder"
 			(at 330.2 167.64 0)
 			(hide yes)
@@
 			)
 		)
-		(property "Footprint" "PoE:TI_0603_1"
+		(property "Footprint" "Capacitor_SMD:C_0603_1608Metric_Pad1.08x0.95mm_HandSolder"
 			(at 231.14 185.42 0)
 			(hide yes)
@@
 			)
 		)
-		(property "Footprint" "PoE:TI_SMB"
+		(property "Footprint" "Diode_SMD:D_SMB_Handsoldering"
 			(at 83.82 175.26 0)
 			(hide yes)
@@
 			)
 		)
-		(property "Footprint" "PoE:TI_SMB"
+		(property "Footprint" "Diode_SMD:D_SMB_Handsoldering"
 			(at 254 175.26 0)
 			(hide yes)
@@
 			)
 		)
-		(property "Footprint" "PoE:TI_0603_2"
+		(property "Footprint" "Resistor_SMD:R_0603_1608Metric_Pad0.98x0.95mm_HandSolder"
 			(at 223.52 170.18 0)
 			(hide yes)
@@
 			)
 		)
-		(property "Footprint" "PoE:TI_SSOT-3"
+		(property "Footprint" "Package_TO_SOT_SMD:SuperSOT-3"
 			(at 241.3 177.8 0)
 			(hide yes)
@@
 			)
 		)
-		(property "Footprint" "PoE:TI_SMB_1"
+		(property "Footprint" "Diode_SMD:D_SMB_Handsoldering"
 			(at 345.44 165.1 0)
 			(hide yes)
@@
 			)
 		)
-		(property "Footprint" "PoE:TI_0603_2"
+		(property "Footprint" "Resistor_SMD:R_0603_1608Metric_Pad0.98x0.95mm_HandSolder"
 			(at 119.38 170.18 0)
 			(hide yes)
@@
 			)
 		)
-		(property "Footprint" "PoE:TI_SMB"
+		(property "Footprint" "Diode_SMD:D_SMB_Handsoldering"
 			(at 162.56 175.26 0)
 			(hide yes)
